File: KiCad/LM5175-DCConverter/LM5175-DCConverter.kicad_pcb (KiCad board)
At the start: 4 copper layers, 57 parts, among them J1 Conn_01x02, J2 Conn_01x02, Q1 CSD18534, Q2 CSD18511, Q3 CSD18534, Q4 CSD18511, U1 LM5175PWP

Commit message: stm32 added
Routing:
- net Vin: vias 3 -> 23
- net SW2: vias 18 -> 14
- net SW1: vias 2 -> 12
- net Isense-: vias 3 -> 27
- net Isense+: vias 2 -> 29
- added copper zone on B.Cu, net Isense+
- added copper zone on In1.Cu, net Isense+
- added copper zone on In2.Cu, net Isense+
- added copper zone on B.Cu, net Isense-
- added copper zone on In1.Cu, net Isense-
- added copper zone on In2.Cu, net Isense-
- added copper zone on B.Cu, net SW1
- added copper zone on In1.Cu, net SW1
- added copper zone on In2.Cu, net SW1

Commit message: MOre PCB work
Parts:
- added C26: 100n, Capacitor_SMD:C_0805_2012Metric, B.Cu at (181.7, 107.2)
- added C27: 100n, Capacitor_SMD:C_0805_2012Metric, B.Cu at (193.2, 97.0)
- added C28: 10u, Capacitor_SMD:C_0805_2012Metric, B.Cu at (193.2, 95.1)
- added C29: 100n, Capacitor_SMD:C_0805_2012Metric, B.Cu at (195.7, 103.4)
- added C30: 1u, Capacitor_SMD:C_0805_2012Metric, B.Cu at (195.7, 105.3)
- added C31: 100n, Capacitor_SMD:C_0805_2012Metric, B.Cu at (195.7, 101.5)
- added C32: 100n, Capacitor_SMD:C_0805_2012Metric, B.Cu at (186.7, 76.8)
- added C33: 100n, Capacitor_SMD:C_0805_2012Metric, B.Cu at (223.5, 56.5)
- added C34: 1u/35V, Capacitor_SMD:C_1206_3216Metric, B.Cu at (97.8, 84.5)
- added C35: 100n, Capacitor_SMD:C_0805_2012Metric, B.Cu at (97.2, 94.6)
- added C36: 1u/20V, Capacitor_SMD:C_1206_3216Metric, B.Cu at (99.7, 94.0)
- added C37: 100n, Capacitor_SMD:C_0805_2012Metric, B.Cu at (99.1, 97.2)
- added C38: 100n, Capacitor_SMD:C_0805_2012Metric, B.Cu at (103.5, 65.4)
- added C39: 4u7/20V, Capacitor_SMD:C_0805_2012Metric, B.Cu at (160.0, 108.6)
- added C40: 4u7, Capacitor_SMD:C_0805_2012Metric, B.Cu at (161.9, 108.6)
- added C41: 100n, Capacitor_SMD:C_0805_2012Metric, B.Cu at (102.2, 71.1)
- added C42: 4u7, Capacitor_SMD:C_0805_2012Metric, B.Cu at (163.8, 108.6)
- added C44: 100n, Capacitor_SMD:C_0805_2012Metric, B.Cu at (195.7, 99.6)
- added C45: 4u7, Capacitor_SMD:C_0805_2012Metric, B.Cu at (172.1, 108.6)
- added D6: LED, LED_SMD:LED_0805_2012Metric, B.Cu at (192.0, 89.2)
- added F1: Fuse, JPFuses:Fuseholder5x20_horiz_open_inline_Type-I, F.Cu at (85.1, 63.5)
- added FL1: BNX025, JPInductors:Filter_Murata_BNX005, F.Cu at (212.7, 74.3)
- added J3: REX128128AYAP3N00000, Connector_FFC-FPC:TE_2-1734839-4_1x24-1MP_P0.5mm_Horizontal, B.Cu at (167.0, 104.1)
- added J4: SWD, Connector_Multicomp:Multicomp_MC9A12-2034_2x10_P2.54mm_Vertical, F.Cu at (222.2, 105.2)
- added L2: L, Inductor_SMD:L_0805_2012Metric, B.Cu at (194.3, 107.2)
- added Q5: IRLML2502, Package_TO_SOT_SMD:SOT-23, F.Cu at (123.8, 95.9)
- added R20: 0, Resistor_SMD:R_0603_1608Metric, B.Cu at (192.5, 93.2)
- added R21: 0, Resistor_SMD:R_0603_1608Metric, B.Cu at (190.6, 93.9)
- added R22: 2m/200mW, Resistor_SMD:R_1206_3216Metric, F.Cu at (104.8, 71.8)
- added R23: 1M, Resistor_SMD:R_1206_3216Metric, B.Cu at (167.6, 108.0)
- added R24: 10k, Resistor_SMD:R_0805_2012Metric, B.Cu at (196.3, 96.0)
- added R25: 10k, Resistor_SMD:R_0805_2012Metric, B.Cu at (196.3, 97.8)
- added R26: 10k, Resistor_SMD:R_0805_2012Metric, B.Cu at (196.2, 88.9)
- added R27: 2k2, Resistor_SMD:R_0805_2012Metric, B.Cu at (188.2, 93.9)
- added R28: 2k2, Resistor_SMD:R_0805_2012Metric, B.Cu at (186.3, 93.9)
- added REF**: REX128128AYAP3N00000, JPDisplays:REX128128AYAP3N00000, B.Cu at (167.0, 81.3)
- added SW1: SW_DIP_x01, Connector_JST:JST_EH_S02B-EH_1x02_P2.50mm_Horizontal, B.Cu at (102.2, 87.0)
- added SW2: SW_DIP_x01, Connector_JST:JST_EH_S02B-EH_1x02_P2.50mm_Horizontal, B.Cu at (113.0, 99.7)
- added SW3: SW_DIP_x01, Button_Switch_SMD:SW_SPST_B3SL-1002P, B.Cu at (216.4, 91.2)
- added U2: INA233, Package_SO:VSSOP-10_3x3mm_P0.5mm, B.Cu at (188.0, 74.3)
- added U3: STM32L051K8Tx, Package_QFP:LQFP-32_7x7mm_P0.8mm, B.Cu at (187.5, 102.1)
- added U4: MCP9800, Package_TO_SOT_SMD:SOT-23-5, B.Cu at (220.3, 56.5)
- added U5: L7815, Package_TO_SOT_SMD:TO-252-2, B.Cu at (92.9, 89.5)
- added U6: L78L33_SOT89, Package_TO_SOT_SMD:SOT-89-3, B.Cu at (103.5, 94.6)
- added U7: MCP9800, Package_TO_SOT_SMD:SOT-23-5, B.Cu at (106.7, 65.4)
- added U8: INA233, Package_SO:VSSOP-10_3x3mm_P0.5mm, B.Cu at (104.8, 72.4)
- moved J2 10.2 mm to (224.2, 76.8)
- moved J1 7.62 mm to (85.1, 76.2)
- moved C1 6.35 mm to (98.4, 73.7)
- moved R19 3.18 mm to (139.7, 95.2)
- moved R3 2.01 mm to (120.7, 98.4)
- moved R5 2.01 mm to (123.8, 98.4)
- moved R18 1.80 mm to (141.0, 97.8), turned to 270 degrees
- moved C25 0.90 mm to (139.1, 97.8)
- moved D1 0.63 mm to (120.0, 101.6)
- moved R4 0.63 mm to (142.9, 101.6), turned to 270 degrees
- moved R6 0.63 mm to (125.7, 101.6)
Connections:
- C1 pad 1: Vin -> Vin+
- C2 pad 1: Vin -> Vin-
- C3 pad 1: Vin -> Vin-
- C4 pad 1: Vin -> Vin-
- D1 pad 2: Vin -> Vin-
- J1 pad 2: Vin -> Net-(F1-Pad1)
- J2 pad 2: Isense- -> Net-(FL1-Pad2)
- Q1 pad 5: Vin -> Vin-
- R3 pad 1: Vin -> Vin-
- U1 pad 3: Vin -> Vin-
Routing:
- net +3V3: track 0.00 -> 172.1 mm, vias 0 -> 5
- net +15V: track 0.00 -> 100.2 mm, vias 0 -> 3
- net CSG: track 73.6 -> 163.2 mm
- net Vin-: track 0.00 -> 57.6 mm, vias 0 -> 19
- net Vin: track 50.8 -> 0.00 mm, vias 23 -> 0
- net SWDIO: track 0.00 -> 41.0 mm, vias 0 -> 1
- net SWCLK: track 0.00 -> 35.0 mm, vias 0 -> 1
- net /D0: track 0.00 -> 30.1 mm, vias 0 -> 2
- net /D1: track 0.00 -> 29.2 mm, vias 0 -> 2
- net Net-(R24-Pad2): track 0.00 -> 28.8 mm
- net /D3: track 0.00 -> 28.6 mm, vias 0 -> 2
- net /D2: track 0.00 -> 28.3 mm, vias 0 -> 2
- net /D4: track 0.00 -> 27.4 mm, vias 0 -> 2
- net /D5: track 0.00 -> 25.8 mm, vias 0 -> 2
- net /!CS: track 0.00 -> 25.2 mm
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- added copper zone on B.Cu, net CSG
- added copper zone on F.Cu, net Net-(F1-Pad1)
- added copper zone on F.Cu, net Net-(FL1-Pad2)
- added copper zone on F.Cu, net Vin+
- added copper zone on F.Cu, net Vin-
- removed copper zone on B.Cu, net Vin
- removed copper zone on F.Cu, net Vin
- removed copper zone on In1.Cu, net Vin
- removed copper zone on In2.Cu, net Vin
Other:
- net class Power added: clearance 0.2, trace_width 1.016, via_dia 1.2, via_drill 0.6
- net class Small added: clearance 0.127, trace_width 0.3048, via_dia 0.6, via_drill 0.4

Commit message: Most of the PCB done
Parts:
- removed C38: 100n, Capacitor_SMD:C_0805_2012Metric
- removed REF**: REX128128AYAP3N00000, JPDisplays:REX128128AYAP3N00000
- removed U4, U7: MCP9800, Package_TO_SOT_SMD:SOT-23-5
- C33: value 100n -> 100u/35V; footprint Capacitor_SMD:C_0805_2012Metric -> Capacitor_SMD:C_Elec_6.3x7.7; moved to F.Cu
- moved C33 123.8 mm to (101.0, 74.1)
- moved D6 20.8 mm to (212.7, 91.2)
- moved R26 17.0 mm to (212.7, 93.2), turned to 180 degrees
- moved C41 13.4 mm to (114.2, 77.3), turned to 0 degrees
- moved U2 10.9 mm to (198.9, 74.7)
- moved U8 10.9 mm to (115.4, 74.7), turned to 180 degrees
- moved C34 10.2 mm to (104.8, 91.9)
- moved C35 10.2 mm to (104.1, 102.0)
- moved C36 10.2 mm to (106.7, 101.4)
- moved U5 10.2 mm to (99.9, 97.0)
- moved U6 10.2 mm to (110.5, 102.0)
- moved C37 10.2 mm to (106.0, 104.6)
- moved C13 10.2 mm to (213.4, 74.1)
- moved C24 10.2 mm to (149.9, 92.5)
- moved R13 10.2 mm to (146.1, 104.0)
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Connections:
- C14 pad 2: CSG -> GNDA
- C15 pad 1: CSG -> GNDA
- C16 pad 1: CSG -> GNDA
- C19 pad 1: CSG -> GNDA
- C20 pad 1: CSG -> GNDA
- C23 pad 1: CSG -> GNDA
- C26 pad 2: CSG -> GNDA
- C27 pad 2: CSG -> GNDA
- C28 pad 2: CSG -> GNDA
- C29 pad 2: CSG -> GNDA
- C30 pad 2: CSG -> GNDA
- C31 pad 2: CSG -> GNDA
- C32 pad 2: CSG -> GNDA
- C33 pad 1: +3V3 -> Vin+
- C34 pad 2: CSG -> GNDA
- C35 pad 2: CSG -> GNDA
- C36 pad 2: CSG -> GNDA
- C37 pad 2: CSG -> GNDA
- C39 pad 1: CSG -> GNDA
- C40 pad 2: CSG -> GNDA
- C41 pad 2: CSG -> GNDA
- C42 pad 2: CSG -> GNDA
- C44 pad 2: CSG -> GNDA
- C45 pad 2: CSG -> GNDA
- J3 pad 1: CSG -> GNDA
- J3 pad 24: CSG -> GNDA
- J3 pad 8: CSG -> GNDA
- J4 pad 10: CSG -> GNDA
- J4 pad 12: CSG -> GNDA
- J4 pad 14: CSG -> GNDA
- J4 pad 18: CSG -> GNDA
- J4 pad 20: CSG -> GNDA
- J4 pad 3: CSG -> GNDA
- J4 pad 4: CSG -> GNDA
- J4 pad 6: CSG -> GNDA
- J4 pad 8: CSG -> GNDA
- Q5 pad 2: CSG -> GNDA
- R14 pad 2: CSG -> GNDA
- R15 pad 2: CSG -> GNDA
- R21 pad 2: CSG -> GNDA
- R23 pad 2: CSG -> GNDA
- R26 pad 2: CSG -> GNDA
- R8 pad 2: CSG -> GNDA
- R9 pad 2: CSG -> GNDA
- SW2 pad 2: CSG -> GNDA
- SW3 pad 2: CSG -> GNDA
- U1 pad 10: CSG -> GNDA
- U1 pad 5: CSG -> GNDA
- U2 pad 1: CSG -> GNDA
- U2 pad 7: CSG -> GNDA
- U3 pad 16: CSG -> GNDA
- U3 pad 25: Net-(U3-Pad25) -> ShutOff
- U3 pad 28: ShutOff -> Net-(U3-Pad28)
- U3 pad 32: CSG -> GNDA
- U5 pad 2: CSG -> GNDA
- U6 pad 2: CSG -> GNDA
- U8 pad 1: CSG -> GNDA
- U8 pad 2: CSG -> GNDA
- U8 pad 7: CSG -> GNDA
Routing:
- net GNDA: track 0.00 -> 182.6 mm, vias 0 -> 14
- net SDA: track 0.00 -> 146.6 mm, vias 0 -> 3
- net SCL: track 0.00 -> 146.4 mm, vias 0 -> 3
- net InaInAlert: track 0.00 -> 124.5 mm, vias 0 -> 4
- net CSG: track 163.2 -> 67.6 mm, vias 2 -> 5
- net ShutOff: track 0.00 -> 84.4 mm, vias 0 -> 1
- net +3V3: track 172.1 -> 244.2 mm, vias 5 -> 10
- net InaOutAlert: track 0.00 -> 29.7 mm, vias 0 -> 2
- net LED: track 0.00 -> 17.7 mm, vias 0 -> 2
- net Vin-: track 57.6 -> 66.2 mm, vias 19 -> 20
- net Vin+: track 0.00 -> 7.29 mm, vias 0 -> 1
- net +15V: track 100.2 -> 106.6 mm
- net Isense-: track 104.3 -> 108.1 mm
- net EN: track 24.1 -> 26.9 mm
- net Net-(D6-Pad1): track 0.00 -> 1.91 mm
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- added copper zone on F.Cu, net +3V3
- added copper zone on B.Cu, net GNDA
- added copper zone on F.Cu, net GNDA
- added copper zone on B.Cu, net Vin+
Other:
- board outline added: 160 x 86 mm
- net class Big added: clearance 0.1778, trace_width 0.6096, via_dia 0.8, via_drill 0.4
- net class Default: clearance 0.2 -> 0.1778; via_dia 0.8 -> 0.6
- net class Power: clearance 0.2 -> 0.1778
- rule trace_clearance: 0.2 -> 0.1778
- board text added: "1. Checklist 2. Vout / Iout - cheatlist 3. Check FFC connector (does pins align?) 4. Tantals instead of electrolites?"
- board text added: "DC/DC Converter v1 JP, 2020.02.11"
- board text added: "Iout | R1||R2 (1206) 8A | 6m5 | 416mW 4A | 12m5 | 200mW 2A | 25m | 100mW 1A | 50m | 50mW"
- board text added: "Vout | L I (R4+R7)/R9 | C12||C13 29.5V I 3u3 I 395.6k/11k | 36uF/50V 12V | 4u7 | 154k/11k | 120uF/20V 5V | 4u7 | 57.8k/11k | 220uF/6.3V"

Commit message: More PCB work
Parts:
- added D7: LED, LED_SMD:LED_0805_2012Metric, B.Cu at (141.0, 82.4)
- added R29: 150, Resistor_SMD:R_0805_2012Metric, F.Cu at (151.1, 106.5)
- added R30: 10k, Resistor_SMD:R_0805_2012Metric, F.Cu at (140.3, 83.0)
- added REF**: MountingHole_3.2mm_M3, MountingHole:MountingHole_3.2mm_M3, F.Cu at (225.4, 111.6)
- added REF**: MountingHole_3.2mm_M3, MountingHole:MountingHole_3.2mm_M3, F.Cu at (84.5, 34.7)
- added REF**: MountingHole_3.2mm_M3, MountingHole:MountingHole_3.2mm_M3, F.Cu at (84.5, 111.6)
- added REF**: MountingHole_3.2mm_M3, MountingHole:MountingHole_3.2mm_M3, F.Cu at (225.4, 34.7)
- added REF**: REX128128AYAP3N00000, JPDisplays:REX128128AYAP3N00000, B.Cu at (177.2, 81.7)
- moved J4 18.9 mm to (213.7, 108.6)
- moved J2 7.73 mm to (225.4, 76.6)
- moved FL1 7.65 mm to (215.3, 74.1)
- moved C13 7.62 mm to (205.7, 74.1)
- moved C12 6.99 mm to (198.8, 74.1)
- moved C32 5.72 mm to (189.1, 75.4)
- moved R1 5.72 mm to (192.4, 67.8)
- moved R2 5.72 mm to (192.4, 71.6)
- moved U2 5.72 mm to (193.2, 74.7)
- moved SW3 5.59 mm to (221.0, 91.9)
- moved C11 3.81 mm to (186.7, 74.1)
- moved C10 3.18 mm to (181.0, 74.1)
- moved C26 2.69 mm to (190.0, 105.7)
- moved C27 2.69 mm to (201.4, 95.6)
- moved C28 2.69 mm to (201.4, 93.7)
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Connections:
- R9 pad 2: GNDA -> Net-(R29-Pad1)
Routing:
- net +3V3: track 244.2 -> 210.9 mm, vias 10 -> 19
- net SWDIO: track 41.0 -> 24.8 mm
- net Net-(D7-Pad1): track 0.00 -> 14.6 mm, vias 0 -> 2
- net SWCLK: track 35.0 -> 22.7 mm
- net GNDA: track 182.6 -> 174.7 mm, vias 14 -> 25
- net Net-(R24-Pad2): track 28.8 -> 22.0 mm
- net Isense+: track 73.4 -> 67.3 mm, vias 29 -> 20
- net Isense-: track 108.1 -> 102.0 mm
- net Vcc: track 25.5 -> 31.5 mm, vias 3 -> 4
- net InaOutAlert: track 29.7 -> 23.9 mm
- net /D7: track 22.4 -> 18.2 mm
- net /D6: track 24.3 -> 20.4 mm
- net InaInAlert: track 124.5 -> 121.0 mm
- net /D5: track 25.8 -> 22.4 mm
- net SCL: track 146.4 -> 143.1 mm
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- added copper zone on In2.Cu, net +3V3
- added copper zone on In1.Cu, net GNDA
- added copper zone on B.Cu, net Net-(F1-Pad1)
- added copper zone on In1.Cu, net Net-(F1-Pad1)
- added copper zone on In2.Cu, net Net-(F1-Pad1)
- added copper zone on In1.Cu, net Vin+
- added copper zone on In2.Cu, net Vin+
Other:
- board size 160 x 86 mm -> 150 x 86 mm
- board text added: "DC/DC Converter v1 JP, 2020.02.16"
- board text added: "DC/DC Enable (open)"
- board text added: "Monitor Power Switch"
- board text added: "Vout | L I (R4+R7)/R9 | C12||C13 29.5V I 3u3 I 400k/11k15 | 36uF/50V 12V | 4u7 | 140k/10k | 120uF/20V 5V | 4u7 | 105k/20k | 220uF/6.3V"
- board text removed: "DC/DC Converter v1 JP, 2020.02.11"
- board text removed: "Vout | L I (R4+R7)/R9 | C12||C13 29.5V I 3u3 I 395.6k/11k | 36uF/50V 12V | 4u7 | 154k/11k | 120uF/20V 5V | 4u7 | 57.8k/11k | 220uF/6.3V"

Commit message: Save before stm32 change
Parts:
- removed REF** (x4): MountingHole_3.2mm_M3, MountingHole:MountingHole_3.2mm_M3
- removed REF**: REX128128AYAP3N00000, JPDisplays:REX128128AYAP3N00000
- added C38: 1u, Capacitor_SMD:C_0805_2012Metric, B.Cu at (199.7, 79.5)
- added C43: 6p, Capacitor_SMD:C_0805_2012Metric, F.Cu at (198.0, 119.8)
- added C46: 100n, Capacitor_SMD:C_0603_1608Metric, F.Cu at (169.7, 109.5)
- added C47: 10u/10V, Capacitor_SMD:C_1206_3216Metric, B.Cu at (109.6, 120.5)
- added H1: MountingHole, MountingHole:MountingHole_3.2mm_M3, F.Cu at (84.8, 34.8)
- added H2: MountingHole, MountingHole:MountingHole_3.2mm_M3, F.Cu at (238.0, 34.2)
- added H3: MountingHole, MountingHole:MountingHole_3.2mm_M3, F.Cu at (237.9, 120.8)
- added H4: MountingHole, MountingHole:MountingHole_3.2mm_M3, F.Cu at (84.0, 120.7)
- added J5: SWD, Connector_PinHeader_2.54mm:PinHeader_1x05_P2.54mm_Horizontal, F.Cu at (231.4, 100.1)
- added Q6: IRLML2502, Package_TO_SOT_SMD:SOT-23, F.Cu at (172.7, 104.9)
- added Q7: BSC340N08NS3, Package_TO_SOT_SMD:TDSON-8-1, F.Cu at (170.3, 72.5)
- added Q8: BSC340N08NS3, Package_TO_SOT_SMD:TDSON-8-1, F.Cu at (157.1, 72.5)
- added Q9: BSC340N08NS3, Package_TO_SOT_SMD:TDSON-8-1, F.Cu at (131.2, 72.5)
- added R31: 100k, Resistor_SMD:R_0805_2012Metric, F.Cu at (130.3, 114.3)
- added R32: 22, Resistor_SMD:R_0805_2012Metric, F.Cu at (174.5, 101.7)
- added R33: 22, Resistor_SMD:R_0805_2012Metric, F.Cu at (176.2, 101.7)
- added R34: 10, Resistor_SMD:R_0805_2012Metric, B.Cu at (119.3, 80.3)
- added R35: 22, Resistor_SMD:R_0805_2012Metric, F.Cu at (177.8, 101.7)
- added R36: 22, Resistor_SMD:R_0805_2012Metric, F.Cu at (179.5, 101.7)
- added R37: 4k7, Resistor_SMD:R_0805_2012Metric, F.Cu at (197.1, 115.3)
- added R38: 2k2, Resistor_SMD:R_0805_2012Metric, F.Cu at (203.5, 116.9)
- added R40: 0, Jumper:SolderJumper-2_P1.3mm_Bridged2Bar_Pad1.0x1.5mm, F.Cu at (116.3, 91.3)
- added U4: MCP9800, Package_TO_SOT_SMD:SOT-23-5, F.Cu at (172.2, 109.9)
- added Y1: 16MHz, Crystal:Crystal_SMD_Abracon_ABM3B-4Pin_5.0x3.2mm, F.Cu at (201.9, 119.8)
- C17: value 100n/X7R/50V -> 1u/X7R/50V
- C26, C27, C32, C35, C37, C41: footprint Capacitor_SMD:C_0805_2012Metric -> Capacitor_SMD:C_0603_1608Metric
- C29: value 100n -> 10n
- C31, C44: footprint Capacitor_SMD:C_0805_2012Metric -> Capacitor_SMD:C_0603_1608Metric; moved to F.Cu
- C36: value 1u/20V -> 4u7/16V
- C39: value 4u7/20V -> 100n; footprint Capacitor_SMD:C_0805_2012Metric -> Capacitor_SMD:C_0603_1608Metric
- C40: value 4u7 -> 100n; footprint Capacitor_SMD:C_0805_2012Metric -> Capacitor_SMD:C_0603_1608Metric
- C42: value 4u7 -> 1u
- C45: value 4u7 -> 6p; moved to F.Cu
- F1: footprint JPFuses:Fuseholder5x20_horiz_open_inline_Type-I -> JPFuses:Fuseholder5x20_horiz_open_big
- J1: value Conn_01x02 -> PowerIN; footprint TerminalBlock:TerminalBlock_bornier-2_P5.08mm -> JPConnectors:XT60PW-M
- J2: value Conn_01x02 -> PowerOUT; footprint TerminalBlock:TerminalBlock_bornier-2_P5.08mm -> JPConnectors:XT60PW-F
- J3: value REX128128AYAP3N00000 -> RVT28AETNWC00; footprint Connector_FFC-FPC:TE_2-1734839-4_1x24-1MP_P0.5mm_Horizontal -> JPConnectors:Hirose_FH12-50S-0.5SH_1x50-1MP_P0.50mm_Horizontal
- J4: value SWD -> TouchPanel; footprint Connector_Multicomp:Multicomp_MC9A12-2034_2x10_P2.54mm_Vertical -> Connector_FFC-FPC:TE_0-1734839-6_1x06-1MP_P0.5mm_Horizontal; moved to B.Cu
- Q1, Q3: value CSD18534 -> BSC340N08NS3
- Q2, Q4: value CSD18511 -> BSC340N08NS3
- R20, R21: value 0 -> 13m/0.5W; footprint Resistor_SMD:R_0603_1608Metric -> Resistor_SMD:R_1206_3216Metric; moved to F.Cu
- R23: value 1M -> 100; footprint Resistor_SMD:R_1206_3216Metric -> Resistor_SMD:R_0805_2012Metric
- R24, R25: footprint Resistor_SMD:R_0805_2012Metric -> Resistor_SMD:R_0603_1608Metric; moved to F.Cu
- R27, R28: value 2k2 -> 4k7; moved to F.Cu
- U3: value STM32L051K8Tx -> STM32L451CEU6; footprint Package_QFP:LQFP-32_7x7mm_P0.8mm -> Package_DFN_QFN:QFN-48-1EP_7x7mm_P0.5mm_EP5.6x5.6mm; moved to F.Cu
- U5: value L7815 -> L78M15
- U6: value L78L33_SOT89 -> LM78M33; footprint Package_TO_SOT_SMD:SOT-89-3 -> Package_TO_SOT_SMD:TO-252-2
- moved C42 59.3 mm to (122.2, 80.3), turned to 0 degrees
- moved D2 54.2 mm to (176.0, 70.7), turned to 90 degrees
- moved D3 45.8 mm to (126.0, 37.0)
- moved C39 35.0 mm to (205.1, 107.4), turned to 180 degrees
- moved R23 34.5 mm to (196.7, 79.5), turned to 180 degrees
- moved C40 26.8 mm to (198.8, 112.0), turned to 90 degrees
- moved C45 26.0 mm to (205.9, 119.8)
- moved D7 21.1 mm to (159.7, 92.1), turned to 90 degrees
- moved R30 20.6 mm to (159.1, 91.4), turned to 0 degrees
- moved R21 19.7 mm to (199.4, 72.7), turned to 180 degrees
- moved C28 19.0 mm to (201.3, 112.7), turned to 90 degrees
- moved R20 16.8 mm to (199.4, 75.0)
- moved C31 16.1 mm to (206.4, 116.0), turned to 270 degrees
- moved R24 16.1 mm to (214.9, 106.9), turned to 90 degrees
- moved D6 15.9 mm to (223.0, 103.3)
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Connections:
- C1 pad 2: CSG -> GND
- C10 pad 2: CSG -> GND
- C11 pad 2: CSG -> GND
- C12 pad 2: CSG -> GND
- C13 pad 2: CSG -> GND
- C14 pad 2: GNDA -> GND
- C15 pad 1: GNDA -> GND
- C16 pad 1: GNDA -> GND
- C17 pad 1: CSG -> GND
- C18 pad 2: CSG -> GND
- C19 pad 1: GNDA -> GND
- C2 pad 2: CSG -> GND
- C20 pad 1: GNDA -> GND
- C23 pad 1: GNDA -> GND
- C26 pad 2: GNDA -> GNDD
- C27 pad 2: GNDA -> GNDD
- C28 pad 2: GNDA -> GNDD
- C29 pad 2: GNDA -> GNDD
- C3 pad 2: CSG -> GND
- C30 pad 2: GNDA -> GNDD
- C31 pad 2: GNDA -> GNDD
- C32 pad 2: GNDA -> GNDD
- C33 pad 2: CSG -> GND
- C34 pad 2: GNDA -> GNDD
- C35 pad 2: GNDA -> GNDD
- C36 pad 2: GNDA -> GNDD
- C37 pad 2: GNDA -> GNDD
- C39 pad 1: GNDA -> +3V3
- C39 pad 2: +15V -> GNDD
- C4 pad 2: CSG -> GND
- C40 pad 1: Net-(C40-Pad1) -> +3V3
- C40 pad 2: GNDA -> GNDD
- C41 pad 2: GNDA -> GNDD
- C42 pad 1: +3V3 -> Net-(C42-Pad1)
- C42 pad 2: GNDA -> Vin-
- C44 pad 2: GNDA -> GNDD
- C45 pad 1: +15V -> Net-(C45-Pad1)
- C45 pad 2: GNDA -> GNDD
- C5 pad 2: CSG -> GND
- C6 pad 2: CSG -> GND
- C7 pad 2: CSG -> GND
- C8 pad 2: CSG -> GND
- C9 pad 2: CSG -> GND
- FL1 pad 2: Net-(FL1-Pad2) -> /PowerOut
- FL1 pad 3: CSG -> GND
- FL1 pad 4: CSG -> GNDPWR
- J1 pad 1: CSG -> GND
- J2 pad 1: CSG -> /PowerOut
- J2 pad 2: Net-(FL1-Pad2) -> GNDPWR
- J3 pad 1: GNDA -> Net-(J3-Pad1)
- J3 pad 10: /!CS -> /LCD_RESET
- J3 pad 11: /!RES -> GNDD
- J3 pad 12: /D_!C -> GNDD
- J3 pad 13: /W -> GNDD
- J3 pad 14: /R -> GNDD
- J3 pad 15: /D0 -> GNDD
- J3 pad 16: /D1 -> GNDD
- J3 pad 17: /D2 -> /D15
- J3 pad 18: /D3 -> /D14
- J3 pad 19: /D4 -> /D13
- J3 pad 2: +15V -> Net-(J3-Pad2)
- J3 pad 20: /D5 -> /D12
- J3 pad 21: /D6 -> /D11
- J3 pad 22: /D7 -> /D10
- J3 pad 23: +15V -> /D9
- J3 pad 24: GNDA -> /D8
- J3 pad 3: Net-(C40-Pad1) -> Net-(J3-Pad3)
- J3 pad 4: +3V3 -> Net-(J3-Pad4)
- J3 pad 5: +3V3 -> Net-(J3-Pad5)
- J3 pad 7: +3V3 -> GNDD
- J3 pad 8: GNDA -> GNDD
- J3 pad 9: Net-(J3-Pad9) -> GNDD
- J4 pad 2: +3V3 -> TP_Reset
- J4 pad 3: GNDA -> TP_Interrupt
- J4 pad 4: GNDA -> SDA
- J4 pad 5: Net-(J4-Pad5) -> SCL
- J4 pad 6: GNDA -> GNDD
- Q5 pad 2: GNDA -> GNDD
- R10 pad 2: CSG -> GND
- R11 pad 2: CSG -> GND
- R14 pad 2: GNDA -> GND
- R15 pad 2: GNDA -> GND
- R17 pad 2: CSG -> GND
- R20 pad 1: +3V3 -> Isense-
- R20 pad 2: Net-(R20-Pad2) -> Isense+
- R21 pad 1: Net-(R20-Pad2) -> Isense-
- R21 pad 2: GNDA -> Isense+
- R23 pad 1: Net-(J3-Pad9) -> Net-(C38-Pad1)
- R23 pad 2: GNDA -> Isense+
- R26 pad 2: GNDA -> GNDD
- R27 pad 2: SDA -> SCL
- R28 pad 2: SCL -> SDA
- R29 pad 2: GNDA -> GND
- R8 pad 2: GNDA -> GND
- SW2 pad 2: GNDA -> GNDD
- SW3 pad 2: GNDA -> GNDD
- U1 pad 10: GNDA -> GND
- U1 pad 22: CSG -> GND
- U1 pad 29: CSG -> GND
- U1 pad 5: GNDA -> GND
- U2 pad 1: GNDA -> GNDD
- U2 pad 10: Isense+ -> Net-(C38-Pad1)
- U2 pad 7: GNDA -> GNDD
- U3 pad 10: /D4 -> Net-(U3-Pad10)
- U3 pad 11: /D5 -> ShutOff
- U3 pad 12: /D6 -> Net-(U3-Pad12)
- U3 pad 13: /D7 -> LED
- U3 pad 14: InaInAlert -> Switch
- U3 pad 15: TempInAlert -> TP_Reset
- U3 pad 16: GNDA -> TP_Interrupt
- U3 pad 17: +3V3 -> InaOutAlert
- U3 pad 18: /R -> /D0
- U3 pad 19: /W -> /D1
- U3 pad 2: Switch -> LCD_BACKGROUD_LED
- U3 pad 20: /D_!C -> /D2
- U3 pad 21: /!RES -> /D10
- U3 pad 22: /!CS -> /D11
- U3 pad 23: SWDIO -> GNDD
- U3 pad 24: SWCLK -> +3V3
- U3 pad 25: ShutOff -> /D12
- U3 pad 26: InaOutAlert -> /D13
- U3 pad 27: TempOutAlert -> /D14
- U3 pad 28: Net-(U3-Pad28) -> /D15
- U3 pad 29: SCL -> /LCD_D_C
- U3 pad 3: LED -> TempAlert
- U3 pad 30: SDA -> SCL
- U3 pad 31: Net-(R20-Pad2) -> SDA
- U3 pad 32: GNDA -> /LCD_WRX
- U3 pad 4: NRST -> InaInAlert
- U3 pad 5: +3.3VADC -> Net-(C43-Pad1)
- U3 pad 6: /D0 -> Net-(R38-Pad1)
- U3 pad 7: /D1 -> NRST
- U3 pad 8: /D2 -> GNDD
- U3 pad 9: /D3 -> +3.3VADC
- U5 pad 2: GNDA -> GNDD
- U6 pad 1: +3V3 -> +15V
- U6 pad 2: GNDA -> GNDD
- U6 pad 3: +15V -> +3V3
- U8 pad 1: GNDA -> GNDD
- U8 pad 10: Vin+ -> Net-(C42-Pad1)
- U8 pad 2: GNDA -> GNDD
- U8 pad 7: GNDA -> GNDD
Routing:
- net GNDA: track 174.7 -> 0.00 mm, vias 25 -> 0
- net +3V3: track 210.9 -> 55.7 mm, vias 19 -> 24
- net GND: track 0.00 -> 118.8 mm, vias 0 -> 12
- net GNDD: track 0.00 -> 114.4 mm, vias 0 -> 36
- net +15V: track 106.6 -> 9.35 mm, vias 3 -> 0
- net CSG: track 67.6 -> 0.00 mm, vias 5 -> 0
- net TempAlert: track 0.00 -> 33.8 mm, vias 0 -> 2
- net LCD_BACKGROUD_LED: track 0.00 -> 33.4 mm, vias 0 -> 2
- net /D11: track 0.00 -> 31.5 mm, vias 0 -> 3
- net /D10: track 0.00 -> 31.3 mm, vias 0 -> 3
- net /D15: track 0.00 -> 29.4 mm, vias 0 -> 1
- net /D14: track 0.00 -> 29.0 mm, vias 0 -> 1
- net /D13: track 0.00 -> 28.7 mm, vias 0 -> 1
- net /D12: track 0.00 -> 28.3 mm, vias 0 -> 1
- net /LCD_RESET: track 0.00 -> 24.4 mm, vias 0 -> 3
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- added copper zone on F.Cu, net /PowerOut
- added copper zone on F.Cu, net GND
- added copper zone on In2.Cu, net GNDA
- added copper zone on B.Cu, net GNDD
- added copper zone on F.Cu, net GNDD
- added copper zone on In1.Cu, net GNDD
- added copper zone on F.Cu, net GNDPWR
- removed copper zone on F.Cu, net +3V3
- removed copper zone on B.Cu, net CSG
- removed copper zone on F.Cu, net CSG
- removed copper zone on F.Cu, net GNDA
- removed copper zone on B.Cu, net Isense+
- removed copper zone on In1.Cu, net Isense+
- removed copper zone on In2.Cu, net Isense+
- removed copper zone on B.Cu, net Isense-
- removed copper zone on In1.Cu, net Isense-
- removed copper zone on In2.Cu, net Isense-
- removed copper zone on B.Cu, net Net-(F1-Pad1)
- removed copper zone on In1.Cu, net Net-(F1-Pad1)
- removed copper zone on In2.Cu, net Net-(F1-Pad1)
- removed copper zone on F.Cu, net Net-(FL1-Pad2)
- removed copper zone on B.Cu, net SW1
- removed copper zone on In1.Cu, net SW1
- removed copper zone on In2.Cu, net SW1
- removed copper zone on B.Cu, net SW2
- removed copper zone on In1.Cu, net SW2
- removed copper zone on In2.Cu, net SW2
- removed copper zone on B.Cu, net Vin+
- removed copper zone on In1.Cu, net Vin+
- removed copper zone on In2.Cu, net Vin+
Other:
- board size 150 x 86 mm -> 162 x 95 mm
- net class Small: via_dia 0.6 -> 0.5; via_drill 0.4 -> 0.3
- board text added: "+3V3"
- board text added: "1. Checklist 4. Tantals instead of electrolites? 5. Vias for pads under devices"
- board text added: "GND"
- board text added: "Iout | R1||R2||* (1206) 8A | 6m5 / 416mW 4A | 12m5 / 200mW 2A | 25m / 100mW 1A | 50m / 50mW"
- board text added: "NRST"
- board text added: "STM32L451CEU6"
- board text added: "SWCLK"
- board text added: "SWD"
- board text added: "SWDIO"
- board text removed: "1. Checklist 2. Vout / Iout - cheatlist 3. Check FFC connector (does pins align?) 4. Tantals instead of electrolites?"
- board text removed: "Iout | R1||R2 (1206) 8A | 6m5 | 416mW 4A | 12m5 | 200mW 2A | 25m | 100mW 1A | 50m | 50mW"
