File: KiCad/LM5175-DCConverter/LM5175-DCConverter.kicad_pcb (KiCad board)
At the start: 4 copper layers, 162 x 95 mm, 126 parts, among them J1 PowerIN, J2 PowerOUT, J3 RVT28AETNWC00, J4 TouchPanel, J5 SWD, Q1 BSC340N08NS3, Q2 BSC340N08NS3, Q3 BSC340N08NS3, Q4 BSC340N08NS3, Q5 IRLML2502, Q6 IRLML2502, Q7 BSC340N08NS3, Q8 BSC340N08NS3, Q9 BSC340N08NS3, SW1 SW_DIP_x01, SW2 SW_DIP_x01, SW3 SW_DIP_x01, U1 LM5175PWP, U2 INA233, U3 STM32L451CEU6, U4 MCP9800, U5 L78M15, U6 LM78M33, U8 INA233, Y1 16MHz

Commit message: First fixes after soldering
Parts:
- removed D3: 950mV/10A, Package_TO_SOT_SMD:TO-252-2_TabPin1
- added D8: 1n4007, Diode_SMD:D_MELF, F.Cu at (100.7, 82.2)
- added L3: 7443630310, JPInductors:L_Wuerth_WE-HCF, F.Cu at (148.6, 53.2)
- added Q10: IRLML2502, Package_TO_SOT_SMD:SOT-23, B.Cu at (135.9, 96.0)
- added R39: 100k, Resistor_SMD:R_0805_2012Metric, B.Cu at (138.4, 94.0)
- added R41: 10k, Resistor_SMD:R_0805_2012Metric, B.Cu at (131.8, 91.8)
- added TP1: TestPoint, TestPoint:TestPoint_THTPad_D1.0mm_Drill0.5mm, F.Cu at (135.9, 64.8)
- added TP2: TestPoint, TestPoint:TestPoint_THTPad_D1.0mm_Drill0.5mm, F.Cu at (161.3, 64.8)
- added TP3: TestPoint, TestPoint:TestPoint_THTPad_D1.0mm_Drill0.5mm, F.Cu at (138.4, 86.4)
- added TP4: TestPoint, TestPoint:TestPoint_THTPad_D1.0mm_Drill0.5mm, F.Cu at (191.8, 72.4)
- added TP5: TestPoint, TestPoint:TestPoint_THTPad_D1.0mm_Drill0.5mm, F.Cu at (212.1, 72.4)
- added TP6: TestPoint, TestPoint:TestPoint_THTPad_D1.0mm_Drill0.5mm, F.Cu at (227.3, 72.4)
- D2: value 500mV/1A/40V -> PowerLED-Good; footprint Diode_SMD:D_SMA -> LED_SMD:LED_0805_2012Metric; moved to B.Cu
- D7: value LED -> PowerLED-Bad
- R30: moved to B.Cu
- SW1, SW2: footprint Connector_JST:JST_EH_S02B-EH_1x02_P2.50mm_Horizontal -> Connector_JST:JST_PH_S2B-PH-K_1x02_P2.00mm_Horizontal
- SW3: footprint Button_Switch_SMD:SW_SPST_B3SL-1002P -> Button_Switch_SMD:SW_SPST_B3S-1000
- U3: value STM32L451CEU6 -> STM32L431CCTx; footprint Package_DFN_QFN:QFN-48-1EP_7x7mm_P0.5mm_EP5.6x5.6mm -> Package_QFP:LQFP-48_7x7mm_P0.5mm
- moved D2 50.5 mm to (130.2, 91.8)
- moved SW1 29.0 mm to (88.1, 107.2)
- moved R30 24.2 mm to (134.9, 91.8), turned to 90 degrees
- moved D7 23.2 mm to (136.5, 91.8)
- moved C34 20.7 mm to (93.1, 108.8), turned to 270 degrees
- moved U5 14.0 mm to (97.7, 111.5), turned to 270 degrees
- moved C47 14.0 mm to (117.2, 108.8), turned to 270 degrees
- moved C37 11.5 mm to (115.4, 108.8), turned to 270 degrees
- moved C35 8.08 mm to (102.2, 108.8), turned to 270 degrees
- moved D4 7.04 mm to (143.3, 93.5), turned to 0 degrees
- moved Q5 6.25 mm to (135.1, 115.8)
- moved R31 6.25 mm to (135.2, 118.1)
- moved SW2 6.15 mm to (127.8, 102.5)
- moved R17 5.67 mm to (159.9, 95.5), turned to 90 degrees
- moved C36 5.50 mm to (104.3, 108.8), turned to 270 degrees
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Connections:
- net Net-(C19-Pad2) renamed /SS
- net Net-(C20-Pad2) renamed /COMP
- net Net-(C23-Pad2) renamed /SLOPE
- net Net-(D7-Pad1) renamed /PGOOD
- net Net-(R14-Pad1) renamed /MODE
- net Net-(R15-Pad1) renamed /RT
- D2 pad 1: Isense+ -> GND
- D2 pad 2: SW2 -> Net-(D2-Pad2)
- J1 pad 1: GND -> Net-(F1-Pad1)
- J1 pad 2: Net-(F1-Pad1) -> GND
- SW1 pad 1: Vin- -> Net-(C34-Pad1)
- SW1 pad 2: Net-(C34-Pad1) -> Vin-
Routing:
- net Vin-: track 67.2 -> 97.4 mm, vias 14 -> 92
- net SW2: track 28.6 -> 47.3 mm, vias 14 -> 127
- net GNDD: track 114.4 -> 101.1 mm, vias 36 -> 66
- net /PGOOD: track 12.1 -> 25.3 mm, vias 1 -> 2
- net GND: track 118.8 -> 108.5 mm, vias 12 -> 128
- net +3V3: track 55.7 -> 64.0 mm
- net Vcc: track 31.7 -> 39.5 mm, vias 3 -> 4
- net SW1: track 34.5 -> 41.8 mm, vias 12 -> 37
- net ShutOff: track 82.4 -> 75.9 mm, vias 2 -> 3
- net Net-(Q10-Pad2): track 0.00 -> 5.54 mm
- net CS: track 30.2 -> 24.8 mm, vias 2 -> 10
- net EN: track 26.9 -> 31.6 mm
- net Net-(C24-Pad2): track 6.01 -> 10.1 mm
- net Isense-: track 102.2 -> 98.3 mm, vias 22 -> 17
- net SCL: track 161.4 -> 163.8 mm
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- added copper zone on B.Cu, net /PowerOut
- added copper zone on In1.Cu, net /PowerOut
- added copper zone on In2.Cu, net /PowerOut
- added copper zone on B.Cu, net CS
- added copper zone on In1.Cu, net CS
- added copper zone on In2.Cu, net CS
- added copper zone on B.Cu, net GND
- added copper zone on In1.Cu, net GND
- added copper zone on In2.Cu, net GND
- added copper zone on B.Cu, net GNDPWR
- added copper zone on In1.Cu, net GNDPWR
- added copper zone on In2.Cu, net GNDPWR
- added copper zone on B.Cu, net Isense+
- added copper zone on In1.Cu, net Isense+
- added copper zone on In2.Cu, net Isense+
- added copper zone on B.Cu, net Isense-
- added copper zone on In1.Cu, net Isense-
- added copper zone on In2.Cu, net Isense-
- added copper zone on B.Cu, net Net-(F1-Pad1)
- added copper zone on In1.Cu, net Net-(F1-Pad1)
- added copper zone on In2.Cu, net Net-(F1-Pad1)
- added copper zone on B.Cu, net SW1
- added copper zone on In1.Cu, net SW1
- added copper zone on In2.Cu, net SW1
- added copper zone on B.Cu, net SW2
- added copper zone on In1.Cu, net SW2
- added copper zone on In2.Cu, net SW2
- added copper zone on B.Cu, net Vin+
- added copper zone on In1.Cu, net Vin+
- added copper zone on In2.Cu, net Vin+
- added copper zone on B.Cu, net Vin-
- added copper zone on In1.Cu, net Vin-
- added copper zone on In2.Cu, net Vin-
- removed copper zone on B.Cu, net GNDA
- removed copper zone on In1.Cu, net GNDA
- removed copper zone on In2.Cu, net GNDA
Other:
- board text added: "C1 C33 - too small Amass - messed up"
- board text added: "DC/DC Converter v1 JP, 2020.08.09"
- board text added: "LM5175PWP"
- board text added: "Power Bad"
- board text added: "Power Good"
- board text added: "STM32L431CCT6"
- board text added: "SW1"
- board text added: "SW2"
- board text removed: "1. Checklist 4. Tantals instead of electrolites? 5. Vias for pads under devices"
- board text removed: "DC/DC Converter v1 JP, 2020.02.16"
- board text removed: "STM32L451CEU6"
