File: KiCad/LM5175-DCConverter/LM5175-DCConverter.kicad_pcb (KiCad board)
At the start: 4 copper layers, 162 x 95 mm, 136 parts, among them J1 PowerIN, J2 PowerOUT, J3 RVT28AETNWC00, J4 TouchPanel, J5 SWD, Q1 BSC340N08NS3, Q10 IRLML2502, Q2 BSC340N08NS3, Q3 BSC340N08NS3, Q4 BSC340N08NS3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

Commit message: Work on pcb v2
Parts:
- removed Q4: BSC340N08NS3, Package_TO_SOT_SMD:TDSON-8-1
- removed the Q9 at (131.2, 72.5)
- added D3: 2A/40V, Diode_SMD:D_SMB, F.Cu at (149.0, 72.0)
- added D9: 1A/40V, Diode_SMD:D_SMB, F.Cu at (182.5, 68.0)
- added Q5: IPD220N06L3 G, Package_TO_SOT_SMD:TO-252-2, F.Cu at (155.0, 70.0)
- added Q6: IPD220N06L3 G, Package_TO_SOT_SMD:TO-252-2, F.Cu at (162.0, 70.0)
- C1, C33: footprint Capacitor_SMD:C_Elec_6.3x7.7 -> Capacitor_SMD:C_Elec_8x6.2
- J2: footprint JPConnectors:XT60PW-F -> JPConnectors:XT60PW-M
- Q1, Q2, Q3, Q7, Q8: value BSC340N08NS3 -> IPD220N06L3 G; footprint Package_TO_SOT_SMD:TDSON-8-1 -> Package_TO_SOT_SMD:TO-252-2
- R22: footprint Resistor_SMD:R_1206_3216Metric -> Resistor_SMD:R_2512_6332Metric
- moved Q2 28.8 mm to (135.5, 70.0)
- moved Q8 19.5 mm to (176.5, 70.0), turned to 270 degrees
- moved Q1 9.03 mm to (128.5, 70.0)
- moved TP6 6.38 mm to (228.8, 78.6)
- moved C33 6.37 mm to (101.6, 82.0)
- moved D8 5.71 mm to (95.0, 82.0)
- moved TP5 5.08 mm to (207.0, 72.4)
- moved J2 4.94 mm to (231.5, 77.5)
- moved L1 4.92 mm to (150.6, 53.5)
- moved L3 4.92 mm to (150.6, 48.7)
- moved C1 4.79 mm to (110.8, 82.0)
- moved TP2 4.75 mm to (162.6, 60.2)
- moved Q10 3.66 mm to (132.6, 94.4)
- moved TP1 3.59 mm to (133.3, 62.2)
- moved C38 3.22 mm to (200.0, 76.3)
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- renumbered Q5 to Q11, Q6 to Q9
Connections:
- D2 pad 1: GND -> Net-(D2-Pad1)
- Q1 pad 1: SW1 -> HDRV1
- Q1 pad 2: SW1 -> Vin-
- Q10 pad 2: Net-(Q10-Pad2) -> GND
- Q10 pad 3: Vcc -> Net-(D2-Pad1)
- Q2 pad 1: SW2 -> HDRV1
- Q2 pad 2: SW2 -> Vin-
- Q2 pad 3: SW2 -> SW1
- Q3 pad 1: CS -> LDRV1
- Q3 pad 2: CS -> SW1
- Q7 pad 1: SW2 -> HDRV2
- Q7 pad 2: SW2 -> Isense+
- Q8 pad 1: CS -> HDRV2
- Q8 pad 2: CS -> Isense+
- Q8 pad 3: CS -> SW2
- R41 pad 1: Net-(Q10-Pad2) -> Vcc
Routing:
- net HDRV2: track 50.5 -> 62.0 mm
- net LDRV1: track 26.8 -> 32.7 mm
- net Net-(Q10-Pad2): track 5.54 -> 0.00 mm
- net LDRV2: track 34.3 -> 39.5 mm
- net SW1: track 41.8 -> 37.5 mm, vias 37 -> 36
- net Net-(D2-Pad1): track 0.00 -> 3.77 mm
- net GNDD: track 101.1 -> 104.5 mm
- net Isense-: track 98.3 -> 101.4 mm, vias 17 -> 20
- net Vcc: track 39.5 -> 42.0 mm, vias 4 -> 3
- net SW2: track 47.3 -> 49.6 mm, vias 127 -> 89
- net Vin-: track 97.4 -> 99.6 mm, vias 92 -> 68
- net Vin+: track 4.21 -> 6.11 mm, vias 30 -> 29
- net InaOutAlert: track 35.6 -> 37.3 mm, vias 1 -> 2
- net SDA: track 168.7 -> 170.5 mm, vias 8 -> 10
- net SCL: track 163.8 -> 165.5 mm, vias 4 -> 6
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- removed copper zone on B.Cu, net /PowerOut
- removed copper zone on In1.Cu, net /PowerOut
- removed copper zone on In2.Cu, net /PowerOut
- removed copper zone on B.Cu, net CS
- removed copper zone on In1.Cu, net CS
- removed copper zone on In2.Cu, net CS
- removed copper zone on B.Cu, net GNDPWR
- removed copper zone on In1.Cu, net GNDPWR
- removed copper zone on In2.Cu, net GNDPWR
- removed copper zone on B.Cu, net Isense+
- removed copper zone on In1.Cu, net Isense+
- removed copper zone on In2.Cu, net Isense+
- removed copper zone on B.Cu, net Isense-
- removed copper zone on In1.Cu, net Isense-
- removed copper zone on In2.Cu, net Isense-
- removed copper zone on B.Cu, net SW2
- removed copper zone on In1.Cu, net SW2
- removed copper zone on In2.Cu, net SW2
Other:
- board text added: "DC/DC Converter v2 JP, 2020.10.31"
- board text added: "more test points? vias quartz"
- board text removed: "C1 C33 - too small Amass - messed up"
- board text removed: "DC/DC Converter v1 JP, 2020.08.09"

Commit message: Last fixes for v2
Parts:
- C26, C30, C39, C40, L2: moved to F.Cu
- C29: value 10n -> 100n; footprint Capacitor_SMD:C_0805_2012Metric -> Capacitor_SMD:C_0603_1608Metric; moved to F.Cu
- moved C31 8.66 mm to (214.0, 110.8)
- moved C30 7.01 mm to (208.4, 116.4), turned to 270 degrees
- moved C29 4.81 mm to (206.8, 116.4), turned to 270 degrees
- moved L2 4.29 mm to (210.2, 116.4), turned to 90 degrees
- moved C26 3.36 mm to (197.4, 115.4), turned to 90 degrees
- moved C40 2.82 mm to (196.0, 113.4)
- moved C39 2.78 mm to (208.7, 106.7), turned to 270 degrees
- moved R37 1.56 mm to (195.7, 116.5), turned to 270 degrees
- moved D6 0.89 mm to (222.6, 104.1)
- moved R26 0.89 mm to (222.6, 106.0)
- moved R38 0.61 mm to (203.6, 118.5)
- moved C43 0.60 mm to (198.0, 121.4)
- moved C45 0.60 mm to (205.9, 121.4)
- moved Y1 0.60 mm to (201.9, 121.4)
- moved R27 0.50 mm to (193.9, 104.0)
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Routing:
- net GNDD: track 104.5 -> 115.2 mm, vias 66 -> 76
- net SDA: track 170.5 -> 176.6 mm
- net +3V3: track 65.3 -> 70.5 mm
- net TempAlert: track 35.2 -> 39.1 mm
- net SCL: track 165.5 -> 167.6 mm
- net +3.3VADC: track 5.89 -> 7.71 mm, vias 1 -> 0
- net ShutOff: track 75.9 -> 77.2 mm
- net Vin-: track 99.6 -> 100.5 mm, vias 68 -> 71
- net /D0: track 29.6 -> 28.9 mm
- net Net-(R38-Pad1): track 3.63 -> 4.38 mm
- net LED: track 19.5 -> 18.7 mm
- net /D1: track 28.6 -> 27.9 mm
- net LCD_BACKGROUD_LED: track 34.0 -> 34.7 mm
- net /D12: track 28.4 -> 29.0 mm
- net NRST: track 33.0 -> 33.7 mm, vias 0 -> 2
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- added copper zone on B.Cu, net /PowerOut
- added copper zone on In1.Cu, net /PowerOut
- added copper zone on In2.Cu, net /PowerOut
- added copper zone on B.Cu, net CS
- added copper zone on In1.Cu, net CS
- added copper zone on In2.Cu, net CS
- added copper zone on B.Cu, net GNDPWR
- added copper zone on In1.Cu, net GNDPWR
- added copper zone on In2.Cu, net GNDPWR
- added copper zone on B.Cu, net Isense+
- added copper zone on In1.Cu, net Isense+
- added copper zone on In2.Cu, net Isense+
- added copper zone on B.Cu, net Isense-
- added copper zone on In1.Cu, net Isense-
- added copper zone on In2.Cu, net Isense-
- added copper zone on B.Cu, net SW2
- added copper zone on In1.Cu, net SW2
- added copper zone on In2.Cu, net SW2
Other:
- board text added: "."
- board text added: "DC/DC Converter v2 JP, 2020.11.4"
- board text removed: "DC/DC Converter v2 JP, 2020.10.31"
- board text removed: "more test points? vias quartz"
