File: KiCad/LM5175-DCConverter/LM5175-DCConverter.sch (KiCad schematic (older format))
At the start: 58 parts, among them J1 Conn_01x02, J2 Conn_01x02, Q1 CSD18534, Q2 CSD18511, Q3 CSD18534, Q4 CSD18511, U1 LM5175PWP

Commit message: stm32 added
Parts:
- added C26, C27, C29, C31, C? (x3): 100n, symbol Device:C
- added C28: 10u, symbol Device:C
- added C30, C? (x4): 1u, symbol Device:C
- added C? (x3): 4u7, symbol Device:C
- added D?: LED, symbol Device:LED
- added J?: Conn_01x24, symbol Connector_Generic:Conn_01x24
- added L2: L, symbol Device:L
- added R20, R21, R? (x2): 10k, symbol Device:R
- added R?: 1M, symbol Device:R
- added U2: INA233, Package_SO:VSSOP-10_3x3mm_P0.5mm, symbol Analog_ADC:INA233
- added U3: STM32L051K8Tx, Package_QFP:LQFP-32_7x7mm_P0.8mm, symbol MCU_ST_STM32L0:STM32L051K8Tx
- added U?: L78L33_SOT89, Package_TO_SOT_SMD:SOT-89-3, symbol Regulator_Linear:L78L33_SOT89
- added U?: L7815, symbol Regulator_Linear:L7815
- gave numbers to parts that had none: 1
Connections:
- net GND: now also C26.2, C27.2, C28.2, C29.2, C30.2, C31.2, C?.1, C?.2, C?.2, C?.2, C?.2, C?.2, C?.2, C?.2, C?.2, C?.2, J?.1 (Pin_1), J?.24 (Pin_24), J?.8 (Pin_8), R21.2, R?.2, U2.7 (GND), U3.16 (VSS), U3.32 (VSS), U?.2 (GND)
- net Isense+: now also U2.10 (Vin+)
- net Isense-: now also U2.8 (Vbus), U2.9 (Vin-)
- new net: R20.2, R21.1, U3.31 (BOOT0)
- new net: C?.1, J?.3 (Pin_3)
- new net: J?.9 (Pin_9), R?.1
- new net: C?.1, U?.1 (IN)
- new net +15V: C?.1, C?.1, C?.1, C?.2, J?.2 (Pin_2), J?.23 (Pin_23), U?.3 (IN), U?.3 (OUT)
- new net +3.3VADC: C29.1, C30.1, L2.2, U3.5 (VDDA)
- new net +3V3: C26.1, C27.1, C28.1, C?.1, C?.1, C?.1, C?.1, J?.4 (Pin_4), J?.5 (Pin_5), J?.6 (Pin_6), J?.7 (Pin_7), L2.1, R20.1, R?.1, R?.1, U2.6 (VS), U3.1 (VDD), U3.17 (VDD), U?.1 (OUT)
- new net D0: J?.15 (Pin_15)
- new net D1: J?.16 (Pin_16)
- new net D2: J?.17 (Pin_17)
- new net D3: J?.18 (Pin_18)
- new net D4: J?.19 (Pin_19)
- new net D5: J?.20 (Pin_20)
- new net D6: J?.21 (Pin_21)
- new net D7: J?.22 (Pin_22)
- new net NRST: C31.1, U3.4 (NRST)
- new net SCL: R?.2, U2.5 (SCL), U3.29 (PB6)
- new net SDA: R?.2, U2.4 (SDA), U3.30 (PB7)
- new net SWCLK: U3.24 (PA14)
- new net SWDIO: U3.23 (PA13)
Other:
- note added: "Address: 100xxxx"
- note added: "REX128128AYAP3N00000"
- moved on the sheet: C1, C10, C11, C12, C13, C14, C15, C16, C17, C18, C19, C2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

Commit message: MOre PCB work
Parts:
- removed C?: 1u, symbol Device:C
- added C33, C38, C41, C44: 100n, Capacitor_SMD:C_0805_2012Metric, symbol Device:C
- added FL1: BNX025, JPInductors:Filter_Murata_BNX005, symbol Filter:BNX025
- added J4: SWD, Connector_Multicomp:Multicomp_MC9A12-2034_2x10_P2.54mm_Vertical, symbol Connector_Generic:Conn_02x10_Odd_Even
- added Q5: IRLML2502, Package_TO_SOT_SMD:SOT-23, symbol Transistor_FET:IRLML2060
- added R22: 2m/200mW, Resistor_SMD:R_1206_3216Metric, symbol Device:R
- added R24, R25, R26: 10k, Resistor_SMD:R_0805_2012Metric, symbol Device:R
- added SW1, SW2: SW_DIP_x01, Connector_JST:JST_EH_S02B-EH_1x02_P2.50mm_Horizontal, symbol Switch:SW_DIP_x01
- added SW3: SW_DIP_x01, Button_Switch_SMD:SW_SPST_B3SL-1002P, symbol Switch:SW_DIP_x01
- added U4, U7: MCP9800, Package_TO_SOT_SMD:SOT-23-5, symbol myLib:MCP9800
- added U8: INA233, Package_SO:VSSOP-10_3x3mm_P0.5mm, symbol Analog_ADC:INA233
- C26, C27, C28, C29, C30, C31: footprint (none) -> Capacitor_SMD:C_0805_2012Metric
- C32, C35, C37, C40, C45: renamed from C?; footprint (none) -> Capacitor_SMD:C_0805_2012Metric
- C34: renamed from C?; value 1u -> 1u/35V; footprint (none) -> Capacitor_SMD:C_1206_3216Metric
- C36: renamed from C?; value 1u -> 1u/20V; footprint (none) -> Capacitor_SMD:C_1206_3216Metric
- C39: renamed from C?; value 4u7 -> 4u7/20V; footprint (none) -> Capacitor_SMD:C_0805_2012Metric
- C42: renamed from C?; value 1u -> 4u7; footprint (none) -> Capacitor_SMD:C_0805_2012Metric
- D6: renamed from D?; footprint (none) -> LED_SMD:LED_0805_2012Metric
- F1: footprint (none) -> JPFuses:Fuseholder5x20_horiz_open_inline_Type-I
- J3: renamed from J?; value Conn_01x24 -> REX128128AYAP3N00000; footprint (none) -> Connector_FFC-FPC:TE_2-1734839-4_1x24-1MP_P0.5mm_Horizontal
- L2: footprint (none) -> Inductor_SMD:L_0805_2012Metric
- R20, R21: value 10k -> 0; footprint (none) -> Resistor_SMD:R_0603_1608Metric
- R23: renamed from R?; footprint (none) -> Resistor_SMD:R_1206_3216Metric
- R27, R28: renamed from R?; value 10k -> 2k2; footprint (none) -> Resistor_SMD:R_0805_2012Metric
- U5: renamed from U?; footprint (none) -> Package_TO_SOT_SMD:TO-252-2
- gave numbers to parts that had none: 1
Connections:
- net +3V3: now also U2.2 (A0), C33.1, C38.1, C41.1, J4.1 (Pin_1), J4.2 (Pin_2), R24.1, U4.1 (VDD), U7.1 (VDD), U8.6 (VS)
- net D0: now also U3.6 (PA0)
- net D1: now also U3.7 (PA1)
- net D2: now also U3.8 (PA2)
- net D3: now also U3.9 (PA3)
- net D4: now also U3.10 (PA4)
- net D5: now also U3.11 (PA5)
- net D6: now also U3.12 (PA6)
- net D7: now also U3.13 (PA7)
- net EN: now also Q5.3 (D), SW2.1
- net GND: now also U2.1 (A1), U5.2 (GND), C33.2, C38.2, C41.2, C44.2, FL1.3 (PSG), FL1.4 (CG), J4.10 (Pin_10), J4.12 (Pin_12), J4.14 (Pin_14), J4.18 (Pin_18), J4.20 (Pin_20), J4.3 (Pin_3), J4.4 (Pin_4), J4.6 (Pin_6), J4.8 (Pin_8), Q5.2 (S), R26.2, SW2.2, SW3.2, U4.2 (GND), U7.2 (GND), U8.1 (A1), U8.2 (A0), U8.7 (GND)
- net Isense-: now also FL1.1 (B); no longer J2.2 (Pin_2)
- net NRST: now also J4.15 (Pin_15)
- net SCL: now also U4.4 (SCLK), U7.4 (SCLK), U8.5 (SCL)
- net SDA: now also U4.5 (SDA), U7.5 (SDA), U8.4 (SDA)
- net SWCLK: now also J4.9 (Pin_9)
- net SWDIO: now also J4.7 (Pin_7)
- net InaInAlert: now reaches U3.14 (PB0)
- net InaInAlert: now also U8.3 (~Alert~)
- net TempInAlert: now reaches U3.15 (PB1)
- net TempInAlert: now also U7.3 (ALERT)
- net R: now reaches U3.18 (PA8)
- net R: now also J3.14 (Pin_14)
- net W: now reaches U3.19 (PA9)
- net W: now also J3.13 (Pin_13)
- net Switch: now reaches U3.2 (PC14)
- net Switch: now also C44.1, R25.2
- net D_!C: now reaches U3.20 (PA10)
- net D_!C: now also J3.12 (Pin_12)
- net !RES: now reaches U3.21 (PA11)
- net !RES: now also J3.11 (Pin_11)
- net !CS: now reaches U3.22 (PA12)
- net !CS: now also J3.10 (Pin_10)
- net InaOutAlert: now reaches U3.26 (PB3)
- net InaOutAlert: now also U2.3 (~Alert~)
- net TempOutAlert: now reaches U3.27 (PB4)
- net TempOutAlert: now also U4.3 (ALERT)
- net ShutOff: now reaches U3.28 (PB5)
- net ShutOff: now also Q5.1 (G)
- net LED: now reaches U3.3 (PC15)
- net LED: now also D6.2 (A)
- net at D6.1 (K): now also R26.1
- net at C34.1, U5.1 (IN): now also SW1.2
- net at F1.1: now also J1.2 (Pin_2)
- net Vin+: now reaches F1.2
- net Vin+: now also C1.1, R22.2, U8.10 (Vin+), U8.8 (Vbus)
- net Vin renamed Vin-
- net Vin-: now also R22.1, SW1.1, U8.9 (Vin-); no longer C1.1, J1.2 (Pin_2)
- new net: FL1.2 (CB), J2.2 (Pin_2)
- new net: R24.2, R25.1, SW3.1
- no-connect marks 0 -> 6
Other:
- note added: "Address: 1000001"
- note added: "INA223, address: 1000000"
- note removed: "Address: 100xxxx"
- moved on the sheet: C1, C26, C27, C28, C29, C30, C31, C34, C35, C36, C37, C39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

Commit message: Most of the PCB done
Parts:
- removed C33, C38: 100n, Capacitor_SMD:C_0805_2012Metric, symbol Device:C
- removed U4, U7: MCP9800, Package_TO_SOT_SMD:SOT-23-5, symbol myLib:MCP9800
- added C33: 100u/35V, Capacitor_SMD:C_Elec_6.3x7.7, symbol Device:CP
- added D?: LED, LED_SMD:LED_0805_2012Metric, symbol Device:LED
- added R?: 0, Resistor_SMD:R_0603_1608Metric, symbol Device:R
Connections:
- net GND: now also C33.2; no longer C14.2, C15.1, C16.1, C19.1, C20.1, C23.1, C26.2, C27.2, C28.2, C29.2, C30.2, C31.2, C32.2, C34.2, C35.2, C36.2, C37.2, C39.1, C40.2, C41.2, C42.2, C44.2, C45.2, J3.1 (Pin_1), J3.24 (Pin_24), J3.8 (Pin_8), J4.10 (Pin_10), J4.12 (Pin_12), J4.14 (Pin_14), J4.18 (Pin_18), J4.20 (Pin_20), J4.3 (Pin_3), J4.4 (Pin_4), J4.6 (Pin_6), J4.8 (Pin_8), Q5.2 (S), R14.2, R15.2, R21.2, R23.2, R26.2, R8.2, R9.2, SW2.2, SW3.2, U1.10 (AGND), U1.5 (DITH), U2.1 (A1), U2.7 (GND), U3.16 (VSS), U3.32 (VSS), U5.2 (GND), U6.2 (GND), U8.1 (A1), U8.2 (A0), U8.7 (GND)
- net ShutOff: now also U3.25 (PA15); no longer U3.28 (PB5)
- net Vcc: now also R?.1
- net Vin+: now also C33.1
- net at U1.17 (PGOOD): now also D?.1 (K)
- new net: D?.2 (A), R?.2
- new net GNDA: C14.2, C15.1, C16.1, C19.1, C20.1, C23.1, C26.2, C27.2, C28.2, C29.2, C30.2, C31.2, C32.2, C34.2, C35.2, C36.2, C37.2, C39.1, C40.2, C41.2, C42.2, C44.2, C45.2, J3.1 (Pin_1), J3.24 (Pin_24), J3.8 (Pin_8), J4.10 (Pin_10), J4.12 (Pin_12), J4.14 (Pin_14), J4.18 (Pin_18), J4.20 (Pin_20), J4.3 (Pin_3), J4.4 (Pin_4), J4.6 (Pin_6), J4.8 (Pin_8), Q5.2 (S), R14.2, R15.2, R21.2, R23.2, R26.2, R8.2, R9.2, SW2.2, SW3.2, U1.10 (AGND), U1.5 (DITH), U2.1 (A1), U2.7 (GND), U3.16 (VSS), U3.32 (VSS), U5.2 (GND), U6.2 (GND), U8.1 (A1), U8.2 (A0), U8.7 (GND)
- no-connect marks 6 -> 7
Other:
- moved on the sheet: F1, J1
Changed lines of the file:
@@
 L Connector_Generic:Conn_01x02 J1
 U 1 1 5E6CAA94
-P 1550 1200
-F 0 "J1" H 1468 875 50  0000 C CNN
-F 1 "Conn_01x02" H 1468 966 50  0000 C CNN
-F 2 "TerminalBlock:TerminalBlock_bornier-2_P5.08mm" H 1550 1200 50  0001 C CNN
-F 3 "~" H 1550 1200 50  0001 C CNN
-	1    1550 1200
+P 1350 1200
+F 0 "J1" H 1268 875 50  0000 C CNN
+F 1 "Conn_01x02" H 1268 966 50  0000 C CNN
+F 2 "TerminalBlock:TerminalBlock_bornier-2_P5.08mm" H 1350 1200 50  0001 C CNN
+F 3 "~" H 1350 1200 50  0001 C CNN
+	1    1350 1200
 	-1   0    0    1
 $EndComp
 Wire Wire Line
-	1750 1100 1950 1100
+	1550 1100 1750 1100
 $Comp
 L power:GND #PWR01
 U 1 1 5E6D7939
-P 1850 1300
-F 0 "#PWR01" H 1850 1050 50  0001 C CNN
-F 1 "GND" H 1855 1127 50  0000 C CNN
-F 2 "" H 1850 1300 50  0001 C CNN
-F 3 "" H 1850 1300 50  0001 C CNN
-	1    1850 1300
-	1    0    0    -1
-$EndComp
-Wire Wire Line
-	1750 1200 1850 1200
-Wire Wire Line
-	1850 1200 1850 1300
+P 1650 1300
+F 0 "#PWR01" H 1650 1050 50  0001 C CNN
+F 1 "GND" H 1655 1127 50  0000 C CNN
+F 2 "" H 1650 1300 50  0001 C CNN
+F 3 "" H 1650 1300 50  0001 C CNN
+	1    1650 1300
+	1    0    0    -1
+$EndComp
+Wire Wire Line
+	1550 1200 1650 1200
+Wire Wire Line
+	1650 1200 1650 1300
 $Comp
 L Connector_Generic:Conn_01x02 J2
@@
 	5200 2850 5200 2750
 Wire Wire Line
-	5200 2750 5350 2750
-Wire Wire Line
 	5350 2750 5350 2850
 $Comp
 L Device:Fuse F1
 U 1 1 5EB4ECD4
-P 2100 1100
-F 0 "F1" H 2160 1146 50  0000 L CNN
-F 1 "Fuse" H 2160 1055 50  0000 L CNN
-F 2 "JPFuses:Fuseholder5x20_horiz_open_inline_Type-I" V 2030 1100 50  0001 C CNN
-F 3 "~" H 2100 1100 50  0001 C CNN
-	1    2100 1100
+P 1900 1100
+F 0 "F1" H 1960 1146 50  0000 L CNN
+F 1 "Fuse" H 1960 1055 50  0000 L CNN
+F 2 "JPFuses:Fuseholder5x20_horiz_open_inline_Type-I" V 1830 1100 50  0001 C CNN
+F 3 "~" H 1900 1100 50  0001 C CNN
+	1    1900 1100
 	0    -1   -1   0
 $EndComp
@@
 $EndComp
 Wire Wire Line
-	2250 1100 2450 1100
+	2050 1100 2200 1100
 Wire Wire Line
 	2950 1100 3200 1100
@@
 	12150 8450 12250 8450
 Connection ~ 12250 8450
-$Comp
-L power:GNDA #PWR0145
-U 1 1 5F5708BD
-P 1800 6450
-F 0 "#PWR0145" H 1800 6200 50  0001 C CNN
-F 1 "GNDA" V 1805 6323 50  0000 R CNN
-F 2 "" H 1800 6450 50  0001 C CNN
-F 3 "" H 1800 6450 50  0001 C CNN
-	1    1800 6450
-	1    0    0    -1
-$EndComp
-$Comp
-L myLib:MCP9800 U7
-U 1 1 5F5969CA
-P 1850 6150
-F 0 "U7" H 1850 6452 40  0000 C CNN
-F 1 "MCP9800" H 1850 6376 40  0000 C CNN
-F 2 "Package_TO_SOT_SMD:SOT-23-5" H 1850 6150 60  0001 C CNN
-F 3 "" H 1850 6150 60  0000 C CNN
-	1    1850 6150
-	1    0    0    -1
-$EndComp
-Text GLabel 2150 6050 2    50   Input ~ 0
-SDA
-Text GLabel 2150 6150 2    50   Input ~ 0
-SCL
-$Comp
-L power:+3.3V #PWR0146
-U 1 1 5F5982CD
-P 1800 5850
-F 0 "#PWR0146" H 1800 5700 50  0001 C CNN
-F 1 "+3.3V" H 1815 6023 50  0000 C CNN
-F 2 "" H 1800 5850 50  0001 C CNN
-F 3 "" H 1800 5850 50  0001 C CNN
-	1    1800 5850
-	1    0    0    -1
-$EndComp
-$Comp
-L Device:C C38
-U 1 1 5F5BDCB1
-P 1350 6100
-F 0 "C38" H 1465 6146 50  0000 L CNN
-F 1 "100n" H 1465 6055 50  0000 L CNN
-F 2 "Capacitor_SMD:C_0805_2012Metric" H 1388 5950 50  0001 C CNN
-F 3 "~" H 1350 6100 50  0001 C CNN
-	1    1350 6100
-	1    0    0    -1
-$EndComp
-$Comp
-L power:+3.3V #PWR0147
-U 1 1 5F5BE481
-P 1350 5950
-F 0 "#PWR0147" H 1350 5800 50  0001 C CNN
-F 1 "+3.3V" H 1365 6123 50  0000 C CNN
-F 2 "" H 1350 5950 50  0001 C CNN
-F 3 "" H 1350 5950 50  0001 C CNN
-	1    1350 5950
-	1    0    0    -1
-$EndComp
-$Comp
-L power:GNDA #PWR0148
-U 1 1 5F5BE88F
-P 1350 6250
-F 0 "#PWR0148" H 1350 6000 50  0001 C CNN
-F 1 "GNDA" V 1355 6123 50  0000 R CNN
-F 2 "" H 1350 6250 50  0001 C CNN
-F 3 "" H 1350 6250 50  0001 C CNN
-	1    1350 6250
-	1    0    0    -1
-$EndComp
-$Comp
-L power:GNDA #PWR0149
-U 1 1 5F5E1D1D
-P 13650 2950
-F 0 "#PWR0149" H 13650 2700 50  0001 C CNN
-F 1 "GNDA" V 13655 2823 50  0000 R CNN
-F 2 "" H 13650 2950 50  0001 C CNN
-F 3 "" H 13650 2950 50  0001 C CNN
-	1    13650 2950
-	1    0    0    -1
-$EndComp
-$Comp
-L myLib:MCP9800 U4
-U 1 1 5F5E1D27
-P 13700 2650
-F 0 "U4" H 13700 2952 40  0000 C CNN
-F 1 "MCP9800" H 13700 2876 40  0000 C CNN
-F 2 "Package_TO_SOT_SMD:SOT-23-5" H 13700 2650 60  0001 C CNN
-F 3 "" H 13700 2650 60  0000 C CNN
-	1    13700 2650
-	1    0    0    -1
-$EndComp
-Text GLabel 14000 2550 2    50   Input ~ 0
-SDA
-Text GLabel 14000 2650 2    50   Input ~ 0
-SCL
-$Comp
-L power:+3.3V #PWR0150
-U 1 1 5F5E1D33
-P 13650 2350
-F 0 "#PWR0150" H 13650 2200 50  0001 C CNN
-F 1 "+3.3V" H 13665 2523 50  0000 C CNN
-F 2 "" H 13650 2350 50  0001 C CNN
-F 3 "" H 13650 2350 50  0001 C CNN
-	1    13650 2350
-	1    0    0    -1
-$EndComp
-$Comp
-L Device:C C33
-U 1 1 5F5E1D3D
-P 13200 2600
-F 0 "C33" H 13315 2646 50  0000 L CNN
-F 1 "100n" H 13315 2555 50  0000 L CNN
-F 2 "Capacitor_SMD:C_0805_2012Metric" H 13238 2450 50  0001 C CNN
-F 3 "~" H 13200 2600 50  0001 C CNN
-	1    13200 2600
-	1    0    0    -1
-$EndComp
-$Comp
-L power:+3.3V #PWR0151
-U 1 1 5F5E1D47
-P 13200 2450
-F 0 "#PWR0151" H 13200 2300 50  0001 C CNN
-F 1 "+3.3V" H 13215 2623 50  0000 C CNN
-F 2 "" H 13200 2450 50  0001 C CNN
-F 3 "" H 13200 2450 50  0001 C CNN
-	1    13200 2450
-	1    0    0    -1
-$EndComp
-$Comp
-L power:GNDA #PWR0152
-U 1 1 5F5E1D51
-P 13200 2750
-F 0 "#PWR0152" H 13200 2500 50  0001 C CNN
-F 1 "GNDA" V 13205 2623 50  0000 R CNN
-F 2 "" H 13200 2750 50  0001 C CNN
-F 3 "" H 13200 2750 50  0001 C CNN
-	1    13200 2750
-	1    0    0    -1
-$EndComp
 Wire Wire Line
 	4050 1950 4050 2000
@@
 Wire Wire Line
 	2350 8000 2250 8000
-Text GLabel 2150 6250 2    50   Input ~ 0
-TempInAlert
 Text GLabel 9300 8650 0    50   Input ~ 0
 InaInAlert
@@
 Text GLabel 3700 7250 0    50   Input ~ 0
 ShutOff
-Text GLabel 9300 9050 0    50   Input ~ 0
+Text GLabel 10400 9250 2    50   Input ~ 0
 ShutOff
-Text GLabel 14000 2750 2    50   Input ~ 0
-TempOutAlert
 Text GLabel 9300 8950 0    50   Input ~ 0
 TempOutAlert
@@
 Wire Wire Line
 	12050 1600 11800 1600
+Connection ~ 11800 1600
+NoConn ~ 9300 9050
+$Comp
+L Device:CP C33
+U 1 1 5E5268A0
+P 2200 1350
+F 0 "C33" H 2318 1396 50  0000 L CNN
+F 1 "100u/35V" H 2318 1305 50  0000 L CNN
+F 2 "Capacitor_SMD:C_Elec_6.3x7.7" H 2238 1200 50  0001 C CNN
+F 3 "~" H 2200 1350 50  0001 C CNN
+	1    2200 1350
+	1    0    0    -1
+$EndComp
+Wire Wire Line
+	2200 1200 2200 1100
+Connection ~ 2200 1100
+Wire Wire Line
+	2200 1100 2450 1100
+Wire Wire Line
+	2200 1500 2200 1600
+Wire Wire Line
+	2200 1600 2450 1600
+Connection ~ 2450 1600
+$Comp
+L Device:R R?
+U 1 1 5E59F0D4
+P 9850 4500
+F 0 "R?" H 9920 4546 50  0000 L CNN
+F 1 "0" H 9920 4455 50  0000 L CNN
+F 2 "Resistor_SMD:R_0603_1608Metric" V 9780 4500 50  0001 C CNN
+F 3 "~" H 9850 4500 50  0001 C CNN
+	1    9850 4500
+	1    0    0    -1
+$EndComp
+$Comp
+L Device:LED D?
+U 1 1 5E59F7DA
+P 9850 4800
+F 0 "D?" V 9889 4683 50  0000 R CNN
+F 1 "LED" V 9798 4683 50  0000 R CNN
+F 2 "LED_SMD:LED_0805_2012Metric" H 9850 4800 50  0001 C CNN
+F 3 "~" H 9850 4800 50  0001 C CNN
+	1    9850 4800
+	0    -1   -1   0
+$EndComp
+Wire Wire Line
+	9050 4250 9850 4250
+Wire Wire Line
+	9850 4250 9850 4350
+Connection ~ 9050 4250
+Wire Wire Line
+	5750 5050 9850 5050
+Wire Wire Line
+	9850 5050 9850 4950
 Wire Bus Line
 	6000 8050 6000 10150
 Wire Bus Line
 	10900 7850 10900 10150
-Connection ~ 11800 1600
 $EndSCHEMATC

Commit message: More PCB work
Parts:
- added R29: 150, Resistor_SMD:R_0805_2012Metric, symbol Device:R
- R30: renamed from R?; value 0 -> 10k; footprint Resistor_SMD:R_0603_1608Metric -> Resistor_SMD:R_0805_2012Metric
- gave numbers to parts that had none: 1
Connections:
- net GNDA: now also R29.2; no longer R9.2
- new net: R29.1, R9.2
Changed lines of the file:
@@
 L power:GNDA #PWR05
 U 1 1 5E491C29
-P 8300 2350
-F 0 "#PWR05" H 8300 2100 50  0001 C CNN
-F 1 "GNDA" H 8305 2177 50  0000 C CNN
-F 2 "" H 8300 2350 50  0001 C CNN
-F 3 "" H 8300 2350 50  0001 C CNN
-	1    8300 2350
+P 8300 2650
+F 0 "#PWR05" H 8300 2400 50  0001 C CNN
+F 1 "GNDA" H 8305 2477 50  0000 C CNN
+F 2 "" H 8300 2650 50  0001 C CNN
+F 3 "" H 8300 2650 50  0001 C CNN
+	1    8300 2650
 	1    0    0    -1
 $EndComp
@@
 Connection ~ 2450 1600
 $Comp
-L Device:R R?
+L Device:R R30
 U 1 1 5E59F0D4
 P 9850 4500
-F 0 "R?" H 9920 4546 50  0000 L CNN
-F 1 "0" H 9920 4455 50  0000 L CNN
-F 2 "Resistor_SMD:R_0603_1608Metric" V 9780 4500 50  0001 C CNN
+F 0 "R30" H 9920 4546 50  0000 L CNN
+F 1 "10k" H 9920 4455 50  0000 L CNN
+F 2 "Resistor_SMD:R_0805_2012Metric" V 9780 4500 50  0001 C CNN
 F 3 "~" H 9850 4500 50  0001 C CNN
 	1    9850 4500
@@
 $EndComp
 $Comp
-L Device:LED D?
+L Device:LED D7
 U 1 1 5E59F7DA
 P 9850 4800
-F 0 "D?" V 9889 4683 50  0000 R CNN
+F 0 "D7" V 9889 4683 50  0000 R CNN
 F 1 "LED" V 9798 4683 50  0000 R CNN
 F 2 "LED_SMD:LED_0805_2012Metric" H 9850 4800 50  0001 C CNN
@@
 Wire Bus Line
 	10900 7850 10900 10150
+$Comp
+L Device:R R29
+U 1 1 5E4AB290
+P 8300 2500
+F 0 "R29" H 8370 2546 50  0000 L CNN
+F 1 "150" H 8370 2455 50  0000 L CNN
+F 2 "Resistor_SMD:R_0805_2012Metric" V 8230 2500 50  0001 C CNN
+F 3 "~" H 8300 2500 50  0001 C CNN
+	1    8300 2500
+	1    0    0    -1
+$EndComp
 $EndSCHEMATC

Commit message: Save before stm32 change
Parts:
- removed J3: REX128128AYAP3N00000, Connector_FFC-FPC:TE_2-1734839-4_1x24-1MP_P0.5mm_Horizontal, symbol Connector_Generic:Conn_01x24
- removed J4: SWD, Connector_Multicomp:Multicomp_MC9A12-2034_2x10_P2.54mm_Vertical, symbol Connector_Generic:Conn_02x10_Odd_Even
- removed U3: STM32L051K8Tx, Package_QFP:LQFP-32_7x7mm_P0.8mm, symbol MCU_ST_STM32L0:STM32L051K8Tx
- removed U6: L78L33_SOT89, Package_TO_SOT_SMD:SOT-89-3, symbol Regulator_Linear:L78L33_SOT89
- added C38: 1u, Capacitor_SMD:C_0805_2012Metric, symbol Device:C
- added C43: 6p, Capacitor_SMD:C_0805_2012Metric, symbol Device:C
- added C46: 100n, Capacitor_SMD:C_0603_1608Metric, symbol Device:C
- added C47: 10u/10V, Capacitor_SMD:C_1206_3216Metric, symbol Device:C
- added H1, H2, H3, H4: MountingHole, MountingHole:MountingHole_3.2mm_M3, symbol Mechanical:MountingHole
- added J3: RVT28AETNWC00, JPConnectors:Hirose_FH12-50S-0.5SH_1x50-1MP_P0.50mm_Horizontal, symbol Connector_Generic:Conn_02x25_Top_Bottom
- added J4: TouchPanel, Connector_FFC-FPC:TE_0-1734839-6_1x06-1MP_P0.5mm_Horizontal, symbol Connector_Generic:Conn_01x06
- added J5: SWD, Connector_PinHeader_2.54mm:PinHeader_1x05_P2.54mm_Horizontal, symbol Connector_Generic:Conn_01x05
- added Q6: IRLML2502, Package_TO_SOT_SMD:SOT-23, symbol Transistor_FET:IRLML2060
- added Q7, Q8, Q9: BSC340N08NS3, Package_TO_SOT_SMD:TDSON-8-1, symbol Transistor_FET:CSD18534Q5A
- added R31: 100k, Resistor_SMD:R_0805_2012Metric, symbol Device:R
- added R32, R33, R35, R36: 22, Resistor_SMD:R_0805_2012Metric, symbol Device:R
- added R34: 10, Resistor_SMD:R_0805_2012Metric, symbol Device:R
- added R37: 4k7, Resistor_SMD:R_0805_2012Metric, symbol Device:R
- added R38: 2k2, Resistor_SMD:R_0805_2012Metric, symbol Device:R
- added R40: 0, Jumper:SolderJumper-2_P1.3mm_Bridged2Bar_Pad1.0x1.5mm, symbol Device:R
- added U3: STM32L451CEU6, Package_DFN_QFN:QFN-48-1EP_7x7mm_P0.5mm_EP5.6x5.6mm, symbol MCU_ST_STM32L4:STM32L451CEUx
- added U4: MCP9800, Package_TO_SOT_SMD:SOT-23-5, symbol myLib:MCP9800
- added U6: LM78M33, Package_TO_SOT_SMD:TO-252-2, symbol Regulator_Linear:LM78M05_TO252
- added Y1: 16MHz, Crystal:Crystal_SMD_Abracon_ABM3B-4Pin_5.0x3.2mm, symbol Device:Crystal_GND24
- C17: value 100n/X7R/50V -> 1u/X7R/50V
- C26, C27, C31, C32, C35, C37, C41, C44: footprint Capacitor_SMD:C_0805_2012Metric -> Capacitor_SMD:C_0603_1608Metric
- C29: value 100n -> 10n
- C36: value 1u/20V -> 4u7/16V
- C39: value 4u7/20V -> 100n; footprint Capacitor_SMD:C_0805_2012Metric -> Capacitor_SMD:C_0603_1608Metric
- C40: value 4u7 -> 100n; footprint Capacitor_SMD:C_0805_2012Metric -> Capacitor_SMD:C_0603_1608Metric
- C42: value 4u7 -> 1u
- C45: value 4u7 -> 6p
- F1: footprint JPFuses:Fuseholder5x20_horiz_open_inline_Type-I -> JPFuses:Fuseholder5x20_horiz_open_big
- J1: value Conn_01x02 -> PowerIN; footprint TerminalBlock:TerminalBlock_bornier-2_P5.08mm -> JPConnectors:XT60PW-M
- J2: value Conn_01x02 -> PowerOUT; footprint TerminalBlock:TerminalBlock_bornier-2_P5.08mm -> JPConnectors:XT60PW-F
- Q1, Q3: value CSD18534 -> BSC340N08NS3
- Q2, Q4: value CSD18511 -> BSC340N08NS3
- R20, R21: value 0 -> 13m/0.5W; footprint Resistor_SMD:R_0603_1608Metric -> Resistor_SMD:R_1206_3216Metric
- R23: value 1M -> 100; footprint Resistor_SMD:R_1206_3216Metric -> Resistor_SMD:R_0805_2012Metric
- R24, R25: footprint Resistor_SMD:R_0805_2012Metric -> Resistor_SMD:R_0603_1608Metric
- R27, R28: value 2k2 -> 4k7
- U5: value L7815 -> L78M15
Connections:
- net +15V: now also U6.1 (VI); no longer C39.2, C45.1
- net +3.3VADC: now also U3.9 (VDDA)
- net +3V3: now also C39.1, C40.1, C46.1, C47.1, J3.40 (Pin_40), J3.41 (Pin_41), J3.42 (Pin_42), J3.6 (Pin_6), J4.1 (Pin_1), J5.1 (Pin_1), R32.2, R33.2, R35.2, R36.2, R37.1, U3.1 (VBAT), U3.24 (VDD), U3.36 (VDDUSB), U3.48 (VDD), U4.1 (VDD), U6.3 (VO); no longer C42.1, R20.1
- net CS: now also Q8.1 (S), Q8.2 (S), Q8.3 (S)
- net D0: now also J3.32 (Pin_32), U3.18 (PB0)
- net D1: now also J3.31 (Pin_31), U3.19 (PB1)
- net D2: now also J3.30 (Pin_30), U3.20 (PB2)
- net D3: now also J3.29 (Pin_29), U3.39 (PB3)
- net D4: now also J3.28 (Pin_28), U3.40 (PB4)
- net D5: now also J3.27 (Pin_27), U3.41 (PB5)
- net D6: now also J3.26 (Pin_26), U3.42 (PB6)
- net D7: now also J3.25 (Pin_25), U3.43 (PB7)
- net GND: now also C14.2, C15.1, C16.1, C19.1, C20.1, C23.1, R14.2, R15.2, R29.2, R8.2, U1.10 (AGND), U1.5 (DITH), R40.2; no longer FL1.4 (CG), J2.1 (Pin_1)
- net HDRV1: now also Q9.4 (G)
- net HDRV2: now also Q7.4 (G)
- net InaInAlert: now also U3.4 (PC15)
- net InaOutAlert: now also U3.17 (PA7)
- net Isense+: now also R20.2, R21.2, R23.2, Q7.5 (D); no longer U2.10 (Vin+)
- net Isense-: now also R20.1, R21.1, C38.2
- net LDRV2: now also Q8.4 (G)
- net LED: now also U3.13 (PA3)
- net NRST: now also J5.5 (Pin_5), U3.7 (NRST)
- net SCL: now also R27.2, J4.5 (Pin_5), U3.30 (PA9), U4.4 (SCLK); no longer R28.2
- net SDA: now also R28.2, J4.4 (Pin_4), U3.31 (PA10), U4.5 (SDA); no longer R27.2
- net SW1: now also Q9.1 (S), Q9.2 (S), Q9.3 (S)
- net SW2: now also Q7.1 (S), Q7.2 (S), Q7.3 (S), Q8.5 (D)
- net SWCLK: now also J5.2 (Pin_2), U3.37 (PA14)
- net SWDIO: now also J5.4 (Pin_4), U3.34 (PA13)
- net ShutOff: now also R31.2, U3.11 (PA1)
- net Switch: now also U3.14 (PA4)
- net Vin+: now also R34.2; no longer U8.10 (Vin+)
- net Vin-: now also C42.2, Q9.5 (D)
- net GNDPWR: now reaches J2.2 (Pin_2)
- net GNDPWR: now also FL1.4 (CG); no longer FL1.2 (CB)
- net at R23.1: now also U2.10 (Vin+), C38.1
- net GNDA renamed GNDD
- net GNDD: now also C39.2, C43.2, C46.2, C47.2, J3.11 (Pin_11), J3.12 (Pin_12), J3.13 (Pin_13), J3.14 (Pin_14), J3.15 (Pin_15), J3.16 (Pin_16), J3.34 (Pin_34), J3.43 (Pin_43), J3.48 (Pin_48), J3.49 (Pin_49), J3.50 (Pin_50), J3.7 (Pin_7), J3.8 (Pin_8), J3.9 (Pin_9), J4.6 (Pin_6), J5.3 (Pin_3), Q6.2 (S), R31.1, R40.1, U3.23 (VSS), U3.35 (VSS), U3.47 (VSS), U3.49 (VSS), U3.8 (VSSA), U4.2 (GND), U6.2 (GND), Y1.2, Y1.4; no longer C14.2, C15.1, C16.1, C19.1, C20.1, C23.1, C39.1, C42.2, R14.2, R15.2, R21.2, R23.2, R29.2, R8.2, U1.10 (AGND), U1.5 (DITH)
- new net: J3.1 (Pin_1), Q6.3 (D)
- new net: J3.2 (Pin_2), R32.1
- new net: J3.3 (Pin_3), R33.1
- new net: J3.4 (Pin_4), R35.1
- new net: J3.5 (Pin_5), R36.1
- new net: C42.1, R34.1, U8.10 (Vin+)
- new net: C43.1, U3.5 (PH0), Y1.1
- new net: C45.1, R38.2, Y1.3
- new net: R38.1, U3.6 (PH1)
- new net D10: J3.22 (Pin_22), U3.21 (PB10)
- new net D11: J3.21 (Pin_21), U3.22 (PB11)
- new net D12: J3.20 (Pin_20), U3.25 (PB12)
- new net D13: J3.19 (Pin_19), U3.26 (PB13)
- new net D14: J3.18 (Pin_18), U3.27 (PB14)
- new net D15: J3.17 (Pin_17), U3.28 (PB15)
- new net D8: J3.24 (Pin_24), U3.45 (PB8)
- new net D9: J3.23 (Pin_23), U3.46 (PB9)
- new net LCD_BACKGROUD_LED: Q6.1 (G), U3.2 (PC13)
- new net LCD_D_C: J3.37 (Pin_37), U3.29 (PA8)
- new net LCD_RDX: J3.35 (Pin_35), U3.33 (PA12)
- new net LCD_RESET: J3.10 (Pin_10), U3.38 (PA15)
- new net LCD_SELECT: J3.38 (Pin_38)
- new net LCD_WRX: J3.36 (Pin_36), U3.32 (PA11)
- new net PowerOut: FL1.2 (CB), J2.1 (Pin_1)
- new net TP_Interrupt: J4.3 (Pin_3), U3.16 (PA6)
- new net TP_Reset: J4.2 (Pin_2), U3.15 (PA5)
- new net TempAlert: R37.2, U3.3 (PC14), U4.3 (ALERT)
- no-connect marks 7 -> 6
Other:
- note added: "STM32L4 ? mA\nLCD n/a ? mA\nLCD LED n/a 80mA\nTouch Panel 00100110 12mA\nINA233 1000000 1mA\nINA233 1000001 1mA\nMCP9800 1001000 1mA"
- note added: "https://webench.ti.com/power-designer/switching-regulator/customize/10?VinMin=22&VinMax=30&O1V=29.5&O1I=8&base_pn=LM5175&AppType=None&Flavor=None&op_TA=20&origin=pf_panel&lang_chosen=en-US&optfactor=3&Topology=Buck_Boost&flavor=None&VoltageOption=None"
- note removed: "REX128128AYAP3N00000"
- moved on the sheet: C1, C14, C2, C26, C27, C28, C29, C3, C30, C31, C33, C4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
