File: KiCad/LM5175-DCConverter/LM5175-DCConverter.sch (KiCad schematic (older format))
At the start: 126 parts, among them J1 PowerIN, J2 PowerOUT, J3 RVT28AETNWC00, J4 TouchPanel, J5 SWD, Q1 BSC340N08NS3, Q2 BSC340N08NS3, Q3 BSC340N08NS3, Q4 BSC340N08NS3, Q5 IRLML2502, Q6 IRLML2502, Q7 BSC340N08NS3, Q8 BSC340N08NS3, Q9 BSC340N08NS3, SW1 SW_DIP_x01, SW2 SW_DIP_x01, SW3 SW_DIP_x01, U1 LM5175PWP, U2 INA233, U3 STM32L451CEU6, U4 MCP9800, U5 L78M15, U6 LM78M33, U8 INA233, Y1 16MHz

Commit message: First fixes after soldering
Parts:
- removed D2: 500mV/1A/40V, Diode_SMD:D_SMA, symbol Device:D_Schottky
- removed D3: 950mV/10A, Package_TO_SOT_SMD:TO-252-2_TabPin1, symbol Device:D_Schottky
- removed U3: STM32L451CEU6, Package_DFN_QFN:QFN-48-1EP_7x7mm_P0.5mm_EP5.6x5.6mm, symbol MCU_ST_STM32L4:STM32L451CEUx
- added D2: PowerLED-Good, LED_SMD:LED_0805_2012Metric, symbol Device:LED
- added D8: 1n4007, Diode_SMD:D_MELF, symbol Device:D
- added L3: 7443630310, JPInductors:L_Wuerth_WE-HCF, symbol Device:L
- added Q10: IRLML2502, Package_TO_SOT_SMD:SOT-23, symbol Transistor_FET:IRLML0030
- added R39: 100k, Resistor_SMD:R_0805_2012Metric, symbol Device:R
- added R41: 10k, Resistor_SMD:R_0805_2012Metric, symbol Device:R
- added TP1, TP2, TP3, TP4, TP5, TP6: TestPoint, TestPoint:TestPoint_THTPad_D1.0mm_Drill0.5mm, symbol Connector:TestPoint
- added U3: STM32L431CCTx, Package_QFP:LQFP-48_7x7mm_P0.5mm, symbol MCU_ST_STM32L4:STM32L431CCTx
- D7: value LED -> PowerLED-Bad
- SW1, SW2: footprint Connector_JST:JST_EH_S02B-EH_1x02_P2.50mm_Horizontal -> Connector_JST:JST_PH_S2B-PH-K_1x02_P2.00mm_Horizontal
- SW3: footprint Button_Switch_SMD:SW_SPST_B3SL-1002P -> Button_Switch_SMD:SW_SPST_B3S-1000
Connections:
- net +3.3VADC: now also U3.9 (VDDA)
- net +3V3: now also U3.1 (VBAT), U3.24 (VDD), U3.36 (VDDUSB), U3.48 (VDD)
- net D0: now also U3.18 (PB0)
- net D1: now also U3.19 (PB1)
- net D10: now also U3.21 (PB10)
- net D11: now also U3.22 (PB11)
- net D12: now also U3.25 (PB12)
- net D13: now also U3.26 (PB13)
- net D14: now also U3.27 (PB14)
- net D15: now also U3.28 (PB15)
- net D2: now also U3.20 (PB2)
- net D3: now also U3.39 (PB3)
- net D4: now also U3.40 (PB4)
- net D5: now also U3.41 (PB5)
- net D6: now also U3.42 (PB6)
- net D7: now also U3.43 (PB7)
- net D8: now also U3.45 (PB8)
- net D9: now also U3.46 (PB9)
- net GND: now also J1.2 (Pin_2), D2.1 (K), D8.2 (A), TP3.1; no longer J1.1 (Pin_1)
- net GNDD: now also U3.23 (VSS), U3.35 (VSS), U3.47 (VSS), U3.8 (VSSA)
- net InaInAlert: now also U3.4 (PC15)
- net InaOutAlert: now also U3.17 (PA7)
- net Isense+: now also TP4.1
- net Isense-: now also TP5.1
- net LCD_BACKGROUD_LED: now also U3.2 (PC13)
- net LCD_D_C: now also U3.29 (PA8)
- net LCD_RDX: now also U3.33 (PA12)
- net LCD_RESET: now also U3.38 (PA15)
- net LCD_WRX: now also U3.32 (PA11)
- net LED: now also U3.13 (PA3)
- net NRST: now also U3.7 (NRST)
- net PowerOut: now also TP6.1
- net SCL: now also U3.30 (PA9)
- net SDA: now also U3.31 (PA10)
- net SW1: now also L3.1, TP1.1
- net SW2: now also L3.2, TP2.1
- net SWCLK: now also U3.37 (PA14)
- net SWDIO: now also U3.34 (PA13)
- net ShutOff: now also U3.11 (PA1)
- net Switch: now also U3.14 (PA4)
- net TP_Interrupt: now also U3.16 (PA6)
- net TP_Reset: now also U3.15 (PA5)
- net TempAlert: now also U3.3 (PC14)
- net Vcc: now also Q10.3 (D), R39.1
- net Vin+: now also D8.1 (K)
- net Vin-: now also SW1.2; no longer SW1.1
- net PGOOD: now reaches D7.1 (K), U1.17 (PGOOD)
- net PGOOD: now also Q10.1 (G), R39.2
- net MODE: now reaches R14.1, U1.4 (MODE)
- net RT: now reaches R15.1, U1.6 (RT/SYNC)
- net SLOPE: now reaches C23.2, U1.7 (SLOPE)
- net SS: now reaches C19.2, U1.8 (SS)
- net COMP: now reaches C20.2, R13.1, U1.9 (COMP)
- net at F1.1: now also J1.1 (Pin_1); no longer J1.2 (Pin_2)
- net at C34.1, U5.1 (IN): now also SW1.1; no longer SW1.2
- net at C43.1, Y1.1: now also U3.5 (PH0)
- net at R38.1: now also U3.6 (PH1)
- new net: D2.2 (A), R41.2
- new net: Q10.2 (S), R41.1
Other:
- note added: "Ven treshold = 1.23V"
- moved on the sheet: C15, C16, C19, C20, C23, C24, C26, C27, C28, C29, C30, C34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

Commit message: Work on pcb v2
Parts:
- removed Q1, Q2, Q3, Q4, Q7, Q8, Q9: BSC340N08NS3, Package_TO_SOT_SMD:TDSON-8-1, symbol Transistor_FET:CSD18534Q5A
- added D3: 2A/40V, Diode_SMD:D_SMB, symbol Device:D_Schottky
- added D9: 1A/40V, Diode_SMD:D_SMB, symbol Device:D_Schottky
- added Q1, Q2, Q3, Q5, Q6, Q7, Q8: IPD220N06L3 G, Package_TO_SOT_SMD:TO-252-2, symbol Device:Q_NMOS_GDS
- C1, C33: footprint Capacitor_SMD:C_Elec_6.3x7.7 -> Capacitor_SMD:C_Elec_8x6.2
- J2: footprint JPConnectors:XT60PW-F -> JPConnectors:XT60PW-M
- R22: footprint Resistor_SMD:R_1206_3216Metric -> Resistor_SMD:R_2512_6332Metric
- renumbered Q5 to Q11, Q6 to Q9
Connections:
- net CS: now also D3.2 (A), Q3.3 (S), Q5.3 (S), Q6.3 (S)
- net GND: now also Q10.2 (S); no longer D2.1 (K)
- net HDRV1: now also Q1.1 (G), Q2.1 (G)
- net HDRV2: now also Q7.1 (G), Q8.1 (G)
- net Isense+: now also D9.1 (K), Q7.2 (D), Q8.2 (D)
- net LDRV1: now also Q3.1 (G)
- net LDRV2: now also Q5.1 (G), Q6.1 (G)
- net SW1: now also D3.1 (K), Q1.3 (S), Q2.3 (S), Q3.2 (D)
- net SW2: now also D9.2 (A), Q5.2 (D), Q6.2 (D), Q7.3 (S), Q8.3 (S)
- net Vcc: now also R41.1; no longer Q10.3 (D)
- net Vin-: now also Q1.2 (D), Q2.2 (D)
- new net: D2.1 (K), Q10.3 (D)
Other:
- note added: "P=8A^2 * 2mA\nP=128mW"
- moved on the sheet: D2, Q10, R41

Commit message: Last fixes for v2
Parts:
- C29: value 10n -> 100n; footprint Capacitor_SMD:C_0805_2012Metric -> Capacitor_SMD:C_0603_1608Metric
Changed lines of the file:
@@
 P 9800 6450
 F 0 "C29" H 9915 6496 50  0000 L CNN
-F 1 "10n" H 9915 6405 50  0000 L CNN
-F 2 "Capacitor_SMD:C_0805_2012Metric" H 9838 6300 50  0001 C CNN
+F 1 "100n" H 9915 6405 50  0000 L CNN
+F 2 "Capacitor_SMD:C_0603_1608Metric" H 9838 6300 50  0001 C CNN
 F 3 "~" H 9800 6450 50  0001 C CNN
 	1    9800 6450
